File: SDI-bridge/PowerSupplies.sch (KiCad schematic (older format))
At the start: 25 parts

Commit message: Add descriptions
Parts:
- added C?: C_33u_0603, antmicro-footprints:0603, symbol antmicroCapacitorspol:C_33u_0603
- added R?: R_105R_0402, antmicro-footprints:0402-res, symbol antmicroResistors0402:R_105R_0402
Connections:
- net GNDA: now also C?.2
- net VPP: now also R?.1
- new net VCO_VDD: C?.1, R?.2
Other:
- note added: "Place close to GS2971A"
- moved on the sheet: C?, R?
