File: SDI-bridge/SDI-bridge.sch (KiCad schematic (older format))
At the start: 26 parts

Commit message: Add descriptions
Parts:
- removed C?: C_33u_0603, antmicro-footprints:0603, symbol antmicroCapacitorspol:C_33u_0603
- removed R?: R_105R_0402, antmicro-footprints:0402-res, symbol antmicroResistors0402:R_105R_0402
Connections:
- net labels added: VCO_VDD
- wire segments 201 -> 206
Other:
- note added: "Place close to GS2971A"
- note added: "We need to choose some of this signals( if needed more space we can change connector to bigger one)"
- moved on the sheet: C?, J?, R?
