File: PowerSupplies.sch (KiCad schematic (older format))
At the start: 27 parts

Commit message: Add todos
Other:
- note added: "TODO: use 3V3 as default input voltage. Use low noise LDO to make 1.2V out of it."
Changed lines of the file:
@@
 EESchema Schematic File Version 4
 LIBS:SDI-bridge-cache
-EELAYER 26 0
+EELAYER 30 0
 EELAYER END
 $Descr A4 11693 8268
@@
 Text Notes 5100 5350 0    79   ~ 0
 Place close to GS2971A
+Text Notes 1450 5550 0    50   ~ 0
+TODO: use 3V3 as default input voltage. Use low noise LDO to make 1.2V out of it.
 $EndSCHEMATC
