File: SDI-bridge.sch (KiCad schematic (older format))
At the start: 107 parts, among them J3 031-70526-21, U1 GS2971A, U2 MAX8902B, Y1 ABM7_27.000MH_D2Y_T

Commit message: Add CrossLink power filtering
Parts:
- removed R? (x2): R_2k37_0402, antmicro-footprints:0402-res, symbol antmicroResistors0402:R_2k37_0402
- added C? (x2): C_4u7_0402, antmicro-footprints:0402-cap, symbol antmicroCapacitors0402:C_4u7_0402
- added C? (x12): C_100n_0402_6V3, antmicro-footprints:0402-cap, symbol antmicroCapacitors0402:C_100n_0402_6V3
- added C? (x4): C_2u2_0402, antmicro-footprints:0402-cap, symbol antmicroCapacitors0402:C_2u2_0402
- added C? (x2): C_1u_0402, antmicro-footprints:0402-cap, symbol antmicroCapacitors0402:C_1u_0402
- added C?: C_2n2_0402, antmicro-footprints:0402-cap, symbol antmicroCapacitors0402:C_2n2_0402
- added FB? (x6): BLM18PG121SN1D, antmicro-footprints:0603, symbol antmicroFerriteBeadsandChips:BLM18PG121SN1D
- added R?: R_0R_0402, antmicro-footprints:0402-res, symbol antmicroResistors0402:R_0R_0402
- added R? (x2): R_4k7_0402, antmicro-footprints:0402-res, symbol antmicroResistors0402:R_4k7_0402
Connections:
- net labels added: GNDGPLL, GNDPLL_DPHY, RST, SCL, SDA, VCCA_DPHY0, VCCA_DPHY1, VCCGPLL, VCCIO_0, VCCIO_1_1, VCCIO_1_2, VCCIO_2_1, VCCIO_2_2, VCCPLL_DPHY0, VCCPLL_DPHY1
- net labels removed: CAM_RST, M1_CAM_SCL, M1_CAM_SDA, M2_CAM_SCL, M2_CAM_SDA
- wire segments 505 -> 631
Other:
- moved on the sheet: C20, C21, C22, C23, C24, C25, C26, C27, C28, C29, C30, C31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

Commit message: Initial component placement and outline definition
Parts:
- removed C? (x3): C_2u2_0402, antmicro-footprints:0402-cap, symbol antmicroCapacitors0402:C_2u2_0402
- removed FB? (x5): BLM18PG121SN1D, antmicro-footprints:0603, symbol antmicroFerriteBeadsandChips:BLM18PG121SN1D
- removed R10, R11, R12, R13, R4, R5, R6, R7, R8, R9: R_0R_0402, antmicro-footprints:0402-res, symbol antmicroResistors0402:R_0R_0402
- added FB1, FB3: BLM18PG121SN1D, antmicro-footprints:0603-res, symbol antmicroFerriteBeadsandChips:BLM18PG121SN1D
- added TP10, TP11, TP12, TP3, TP4, TP5, TP6, TP7, TP8, TP9: TP_SMD_0_75MM, antmicro-footprints:Testpoint_smd_0_75mm, symbol antmicroTestPoints:TP_SMD_0_75MM
- FB2: renamed from FB?; footprint antmicro-footprints:0603 -> antmicro-footprints:0603-res
- U3: renamed from U?; footprint (none) -> antmicro-footprints:QFN-16_EP_4x4_Pitch0.65mm
- U4: renamed from U?; footprint (none) -> antmicro-footprints:BGA-80pin_ckfBGA80_7.0x7.0mm
- gave numbers to parts that had none: 42
Connections:
- net labels removed: DOUT0, DOUT1, DOUT2, DOUT3, DOUT4, DOUT5, DOUT6, DOUT7, DOUT8, DOUT9, DOUT[9:0]
- wire segments 631 -> 606

Commit message: Expose DPHY1 at FFC connector
Parts:
- added J4, J5: MC-HVT1-S04-G, antmicro-footprints:PinHeader_1x4_P1.27mm_Drill.7mm, symbol antmicroRectangularConnectorsHeadersMalePins:MC-HVT1-S04-G
- added R10, R11, R12, R13, R49, R50, R51, R52, R53, R54, R55, R56, R57, R58, R59, R6, R60, R61, R62, R65, R67, R68, R69, R70, R8, R9: R_0R_0402, antmicro-footprints:0402-res, symbol antmicroResistors0402:R_0R_0402
- added R4, R5, R63, R64, R66, R7: R_2k37_0402, antmicro-footprints:0402-res, symbol antmicroResistors0402:R_2k37_0402
- added TP13, TP14, TP17, TP18: TP_SMD1MM, antmicro-footprints:Testpoint_smd_1mm, symbol antmicroTestPoints:TP_SMD1MM
- added U5: SC18IS602BIPW, antmicro-footprints:SC18IS602B, symbol antmicroInterfaceDriversReceiversTransceivers:SC18IS602BIPW
Connections:
- net labels added: DPHY0_CLK_N, DPHY0_CLK_P, DPHY0_D0_N, DPHY0_D0_P, DPHY0_D1_N, DPHY0_D1_P, DPHY0_D2_N, DPHY0_D2_P, DPHY0_D3_N, DPHY0_D3_P, DPHY1_CLK_N, DPHY1_CLK_P, DPHY1_D0_N, DPHY1_D0_P, DPHY1_D1_N, DPHY1_D1_P, DPHY1_D2_N, DPHY1_D2_P, DPHY1_D3_N, DPHY1_D3_P, MIPI0_CLK_N, MIPI0_CLK_P, MIPI0_D0_N, MIPI0_D0_P, MIPI0_D1_N, MIPI0_D1_P, MIPI0_D2_N, MIPI0_D2_P, MIPI0_D3_N, MIPI0_D3_P, MIPI1_CLK_N, MIPI1_CLK_P, MIPI1_D0_N, MIPI1_D0_P, MIPI1_D1_N, MIPI1_D1_P, MIPI1_D2_N, MIPI1_D2_P, MIPI1_D3_N, MIPI1_D3_P, SCL_CL, SCL_GS, SDA_CL, SDA_GS, VCCA_DPHY, VCCIO
- net labels removed: MIPI_CLK_N, MIPI_CLK_P, MIPI_D0_N, MIPI_D0_P, MIPI_D1_N, MIPI_D1_P, MIPI_D2_N, MIPI_D2_P, MIPI_D3_N, MIPI_D3_P, VCCA_DPHY0, VCCA_DPHY1, VCCIO_0, VCCIO_1_1, VCCIO_1_2, VCCIO_2_1, VCCIO_2_2, VCCPLL_DPHY0, VCCPLL_DPHY1
- wire segments 606 -> 712
- no-connect marks 0 -> 8
Other:
- note added: "CrossLink Power Filtering"
- note added: "Do we need enable signals controlled from FPGA?"
- note added: "GS Power Filtering"
- note added: "I2C exposed at goldpins"
- note added: "I2C to SPI bridge"
- note added: "MIPI conector"
- note added: "Second option to connect I2C"
- note added: "Unused Audio chanels"
- note removed: "Power Filtering"
- moved on the sheet: C64, C66, R26, R27, R28, R29, R43, TP15

Commit message: Update component placement
Parts:
- removed J2: WE_68715014522, antmicro-footprints:WE_68715014522, symbol antmicroFCCConnectors:WE_68715014522
- removed R4, R46, R48, R5: R_2k37_0402, antmicro-footprints:0402-res, symbol antmicroResistors0402:R_2k37_0402
- removed R47, R67, R68, R69, R70: R_0R_0402, antmicro-footprints:0402-res, symbol antmicroResistors0402:R_0R_0402
- added J3: WE_68715014522_ONE-SIDE, antmicro-footprints:WE_68715014522_ONE-SIDE, symbol antmicroFCCConnectors:WE_68715014522_ONE-SIDE
- added R31, R37, R38, R39, R40, R41, R42: R_0R_0402, antmicro-footprints:0402-res, symbol antmicroResistors0402:R_0R_0402
- renumbered C2 to C10, C28 to C11, C29 to C12, C30 to C13, C31 to C14, C3 to C15, C32 to C16, C33 to C17, C37 to C18, C5 to C19, C20 to C2, C6 to C20, C38 to C21, C39 to C22, C40 to C23, C7 to C24, C8 to C25, C41 to C26, C42 to C27, C10 to C28, C11 to C29, C21 to C3, C43 to C30, C44 to C31, C12 to C32, C13 to C33, C45 to C34, C9 to C35, C46 to C36, C47 to C37, C53 to C38, C61 to C39, C22 to C4, C57 to C40, C48 to C41, C62 to C42, C34 to C43, C58 to C44, C64 to C45, C49 to C46, C66 to C47, C63 to C48, C59 to C49, C23 to C5, C67 to C51, C65 to C52, C60 to C53, C51 to C54, C35 to C55, C36 to C56, C52 to C57, C4 to C58, C14 to C59, C24 to C6, C15 to C60, C16 to C61, C17 to C62, C18 to C63, C19 to C64, C25 to C7, C26 to C8, C27 to C9, J3 to J2, R17 to R10, R18 to R11, R19 to R12, R20 to R13, R21 to R14, R22 to R15, R23 to R16, R26 to R17, R27 to R18, R28 to R19, R29 to R20, R35 to R21, R36 to R22, R37 to R23, R30 to R24, R34 to R25, R43 to R26, R40 to R27, R41 to R28, R42 to R29, R33 to R30, R38 to R32, R24 to R33, R39 to R34, R44 to R35, R45 to R36, R25 to R4, R6 to R43, R53 to R44, R54 to R45, R55 to R46, R56 to R47, R57 to R48, R58 to R49, R31 to R5, R59 to R50, R60 to R51, R61 to R52, R62 to R53, R8 to R54, R9 to R55, R10 to R56, R11 to R57, R12 to R58, R13 to R59, R32 to R6, R49 to R60, R50 to R61, R51 to R62, R52 to R63, R7 to R64, R63 to R65, R64 to R66, R65 to R67, R66 to R68, R14 to R7, R15 to R8, R16 to R9, TP6 to TP10, TP7 to TP11, TP8 to TP12, TP9 to TP13, TP10 to TP14, TP11 to TP15, TP12 to TP16, TP15 to TP17, TP13 to TP3, TP14 to TP4, TP17 to TP5, TP16 to TP6, TP3 to TP7, TP4 to TP8, TP5 to TP9, U2 to U1, U1 to U2
Connections:
- net labels added: CD_VDD, IO_VDD, LOCKED_IN, SCL1, SCL2, SDA1, SDA2, VCC_IO
- net labels removed: +VSW, SCL, SDA
- wire segments 712 -> 710
Other:
- note added: "CrossLink and Semtech at same I2C Line"
- note added: "DNP if one I2C used"
- note added: "Locked from GS connected to CrossLink"
- note removed: "DNP"
- note removed: "Second option to connect I2C"
- moved on the sheet: D1, R33, R44, R45, R46, R47, R48, R49, R50, R51, R52, R53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

Commit message: Schematic changes after design review
Parts:
- added C65: C_10n_0402, antmicro-footprints:0402-cap, symbol antmicroCapacitors0402:C_10n_0402
- added R69, R70, R71, R72, R73, R74: R_0R_0402, antmicro-footprints:0402-res, symbol antmicroResistors0402:R_0R_0402
Connections:
- wire segments 710 -> 734
- no-connect marks 8 -> 4
Other:
- note added: "DNP"
- note added: "TODO: add a possibility to put crosslink in RST state"
- note added: "TODO: add pull-ups / pull-downs for initial states"
- note added: "TODO: connect CDONE to LED?"
- moved on the sheet: C18, C22, C36, C45, J1, R17, R18, R19, R20, R26

Commit message: Add routing on 6 layers
Parts:
- added D2: LG_L29K-G2J1-24-Z, antmicro-footprints:LED_0603, symbol antmicroLEDIndicationDiscrete:LG_L29K-G2J1-24-Z
- added R75, R76, R77, R78, R79, R80, R81, R82, R83, R84, R85, R86, R87, R89, R90, R91: R_0R_0402, antmicro-footprints:0402-res, symbol antmicroResistors0402:R_0R_0402
- added R88: R_100R_0402, antmicro-footprints:0402-res, symbol antmicroResistors0402:R_100R_0402
- added TP19, TP20, TP21, TP22: TP_SMD1MM, antmicro-footprints:Testpoint_smd_1mm, symbol antmicroTestPoints:TP_SMD1MM
Connections:
- net labels added: CDONE, LOCKED_CL
- net labels removed: CD_VDD, GND, LOCKED_IN, VCCIO
- wire segments 734 -> 771
Other:
- note removed: "TODO: add a possibility to put crosslink in RST state"
- note removed: "TODO: connect CDONE to LED?"
- moved on the sheet: R28

Commit message: Fix inner layer clearance and tracks width
Parts:
- C1, C15: footprint antmicro-footprints:0603-cap -> SDI-bridge-footprints:0603-cap; symbol antmicroCapacitors0603:C_10u_0603 -> SDI-bridge:C_10u_0603
- C10, C11, C12, C13, C14, C16, C17, C18, C19, C2, C20, C21, C22, C3, C32, C33, C34, C36, C4, C5, C6, C65, C7, C8, C9: footprint antmicro-footprints:0402-cap -> SDI-bridge-footprints:0402-cap; symbol antmicroCapacitors0402:C_10n_0402 -> SDI-bridge:C_10n_0402
- C23, C31, C42, C52: footprint antmicro-footprints:0402-cap -> SDI-bridge-footprints:0402-cap; symbol antmicroCapacitors0402:C_4u7_0402 -> SDI-bridge:C_4u7_0402
- C24, C25, C26, C28, C29, C30, C35, C45, C47, C55, C56, C62: footprint antmicro-footprints:0402-cap -> SDI-bridge-footprints:0402-cap; symbol antmicroCapacitors0402:C_1u_0402 -> SDI-bridge:C_1u_0402
- C27: footprint antmicro-footprints:0402-res -> SDI-bridge-footprints:0402-res; symbol antmicroCapacitors0402:C_5n6_0402 -> SDI-bridge:C_5n6_0402
- C37: footprint antmicro-footprints:0402-cap -> SDI-bridge-footprints:0402-cap; symbol antmicroCapacitors0402:C_2n2_0402 -> SDI-bridge:C_2n2_0402
- C38: footprint antmicro-footprints:0402-cap -> SDI-bridge-footprints:0402-cap; symbol antmicroCapacitors0402:C_2u2_0402 -> SDI-bridge:C_2u2_0402
- C39, C40, C41, C44, C46, C48, C49, C50, C51, C53, C54, C57: footprint antmicro-footprints:0402-cap -> SDI-bridge-footprints:0402-cap; symbol antmicroCapacitors0402:C_100n_0402_6V3 -> SDI-bridge:C_100n_0402_6V3
- C43: footprint antmicro-footprints:0603-res -> SDI-bridge-footprints:0603-res; symbol antmicroCapacitors0603:C_6n2_0603 -> SDI-bridge:C_6n2_0603
- C58: footprint antmicro-footprints:0603-cap -> SDI-bridge-footprints:0603-cap; symbol antmicroCapacitorspol:C_33u_0603 -> SDI-bridge:C_33u_0603
- C59, C60: footprint antmicro-footprints:0402-res -> SDI-bridge-footprints:0402-res; symbol antmicroCapacitors0402:C_16p_0402 -> SDI-bridge:C_16p_0402
- C61, C64: footprint antmicro-footprints:0402-cap -> SDI-bridge-footprints:0402-cap; symbol antmicroCapacitors0402:C_470n_0402 -> SDI-bridge:C_470n_0402
- C63: footprint antmicro-footprints:0402-cap -> SDI-bridge-footprints:0402-cap; symbol antmicroCapacitors0402:C_47n_0402 -> SDI-bridge:C_47n_0402
- D1, D2: footprint antmicro-footprints:LED_0603 -> SDI-bridge-footprints:LED_0603; symbol antmicroLEDIndicationDiscrete:LG_L29K-G2J1-24-Z -> SDI-bridge:LG_L29K-G2J1-24-Z
- FB1, FB2, FB3: footprint antmicro-footprints:0603-res -> SDI-bridge-footprints:0603-res; symbol antmicroFerriteBeadsandChips:BLM18PG121SN1D -> SDI-bridge:BLM18PG121SN1D
- J1, J2: footprint antmicro-footprints:BNC_Edge_Conn -> SDI-bridge-footprints:BNC_Edge_Conn; symbol antmicroCoaxialConnectorsRF:031-70526-21 -> SDI-bridge:031-70526-21
- J3: footprint antmicro-footprints:WE_68715014522_ONE-SIDE -> SDI-bridge-footprints:WE_68715014522_ONE-SIDE; symbol antmicroFCCConnectors:WE_68715014522_ONE-SIDE -> SDI-bridge:WE_68715014522_ONE-SIDE
- J4, J5: footprint antmicro-footprints:PinHeader_1x4_P1.27mm_Drill.7mm -> SDI-bridge-footprints:PinHeader_1x4_P1.27mm_Drill.7mm; symbol antmicroRectangularConnectorsHeadersMalePins:MC-HVT1-S04-G -> SDI-bridge:MC-HVT1-S04-G
- N1: footprint antmicro-footprints:antmicro-logo_scaled_20mm -> SDI-bridge-footprints:antmicro-logo_scaled_20mm; symbol antmicroMechanicalParts:antmicro_logo -> SDI-bridge:antmicro_logo
- R1, R2, R3: footprint antmicro-footprints:0402-res -> SDI-bridge-footprints:0402-res; symbol antmicroResistors0402:R_22R_0402 -> SDI-bridge:R_22R_0402
- R10, R11, R12, R13, R14, R15, R16, R21, R22, R23, R24, R25, R26, R31, R32, R34, R37, R38, R39, R40, R41, R42, R43, R44, R45, R46, R47, R48, R49, R50, R51, R52, R53, R54, R55, R56, R57, R58, R59, R60, R61, R62, R63, R67, R69, R7, R70, R71, R72, R73, R74, R75, R76, R77, R78, R79, R8, R80, R81, R82, R83, R84, R85, R86, R87, R89, R9, R90, R91: footprint antmicro-footprints:0402-res -> SDI-bridge-footprints:0402-res; symbol antmicroResistors0402:R_0R_0402 -> SDI-bridge:R_0R_0402
- R17, R18, R19, R20, R27, R28: footprint antmicro-footprints:0603-res -> SDI-bridge-footprints:0603-res; symbol antmicroResistors0603:R_75R_0603 -> SDI-bridge:R_75R_0603
- R29: footprint antmicro-footprints:0402-res -> SDI-bridge-footprints:0402-res; symbol antmicroResistors0402:R_37R4_0402 -> SDI-bridge:R_37R4_0402
- R30: footprint antmicro-footprints:0402-res -> SDI-bridge-footprints:0402-res; symbol antmicroResistors0402:R_105R_0402 -> SDI-bridge:R_105R_0402
- R33, R88: footprint antmicro-footprints:0402-res -> SDI-bridge-footprints:0402-res; symbol antmicroResistors0402:R_100R_0402 -> SDI-bridge:R_100R_0402
- R35, R36: footprint antmicro-footprints:0402-res -> SDI-bridge-footprints:0402-res; symbol antmicroResistors0402:R_4k7_0402 -> SDI-bridge:R_4k7_0402
- R4: footprint antmicro-footprints:0402-res -> SDI-bridge-footprints:0402-res; symbol antmicroResistors0402:R_750R_0402 -> SDI-bridge:R_750R_0402
- R5, R6: footprint antmicro-footprints:0402-res -> SDI-bridge-footprints:0402-res; symbol antmicroResistors0402:R_120k_0402 -> SDI-bridge:R_120k_0402
- R64, R65, R66, R68: footprint antmicro-footprints:0402-res -> SDI-bridge-footprints:0402-res; symbol antmicroResistors0402:R_2k37_0402 -> SDI-bridge:R_2k37_0402
- TP1, TP17, TP18, TP19, TP2, TP20, TP21, TP22, TP3, TP4, TP5, TP6: footprint antmicro-footprints:Testpoint_smd_1mm -> SDI-bridge-footprints:Testpoint_smd_1mm; symbol antmicroTestPoints:TP_SMD1MM -> SDI-bridge:TP_SMD1MM
- TP10, TP11, TP12, TP13, TP14, TP15, TP16, TP7, TP8, TP9: footprint antmicro-footprints:Testpoint_smd_0_75mm -> SDI-bridge-footprints:Testpoint_smd_0_75mm; symbol antmicroTestPoints:TP_SMD_0_75MM -> SDI-bridge:TP_SMD_0_75MM
- U1: footprint antmicro-footprints:TDFN2x2 -> SDI-bridge-footprints:TDFN2x2; symbol antmicroPMICVoltageRegulatorsLinear:MAX8902B -> SDI-bridge:MAX8902B
- U2: footprint antmicro-footprints:BGA100_11x11mm -> SDI-bridge-footprints:BGA100_11x11mm; symbol antmicroInterfaceControllers:GS2971A -> SDI-bridge:GS2971A
- U3: footprint antmicro-footprints:QFN-16_EP_4x4_Pitch0.65mm -> SDI-bridge-footprints:QFN-16_EP_4x4_Pitch0.65mm; symbol antmicroInterfaceControllers:GS2988 -> SDI-bridge:GS2988
- U4: footprint antmicro-footprints:BGA-80pin_ckfBGA80_7.0x7.0mm -> SDI-bridge-footprints:BGA-80pin_ckfBGA80_7.0x7.0mm; symbol antmicroBGAchips:CrossLink_LIF-MD6000-6JMG80I -> SDI-bridge:CrossLink_LIF-MD6000-6JMG80I
- U5: footprint antmicro-footprints:SC18IS602B -> SDI-bridge-footprints:SC18IS602B; symbol antmicroInterfaceDriversReceiversTransceivers:SC18IS602BIPW -> SDI-bridge:SC18IS602BIPW
- Y1: footprint antmicro-footprints:ABM7_OSC -> SDI-bridge-footprints:ABM7_OSC; symbol antmicroOscillators:ABM7_27.000MH_D2Y_T -> SDI-bridge:ABM7_27.000MH_D2Y_T

Commit message: Add I2S connector and GND planes
Parts:
- added J6: MC-HVT1-S04-G, antmicro-footprints:PinHeader_1x4_P1.27mm_Drill.7mm, symbol antmicroRectangularConnectorsHeadersMalePins:MC-HVT1-S04-G
Connections:
- wire segments 771 -> 775
Other:
- note added: "I2S connector"
