File: SDI-bridge.sch (KiCad schematic (older format))
At the start: 196 parts, among them J1 031-70526-21, J2 031-70526-21, J3 WE_68715014522_ONE-SIDE, J4 MC-HVT1-S04-G, J5 MC-HVT1-S04-G, J6 MC-HVT1-S04-G, U1 MAX8902B, U2 GS2971A, U3 GS2988, U4 CrossLink_LIF-MD6000-6JMG80I, U5 SC18IS602BIPW, Y1 ABM7_27.000MH_D2Y_T

Commit message: Schematic updates
Parts:
- R32, R34: DNP (none) -> 1
Connections:
- wire segments 775 -> 777
Other:
- note added: "Cross Link"
- note added: "I2C pull-ups"
- note removed: "Do we need enable signals controlled from FPGA?"
- note removed: "Locked from GS connected to CrossLink"
- note removed: "SPI"
- note removed: "TODO: add pull-ups / pull-downs for initial states"

Commit message: Add LED indicators and swap pin numbers of BNC connectors
Parts:
- added D? (x2): LG_L29K-G2J1-24-Z, SDI-bridge-footprints:LED_0603, symbol SDI-bridge:LG_L29K-G2J1-24-Z
- added R? (x2): R_100R_0402, SDI-bridge-footprints:0402-res, symbol SDI-bridge:R_100R_0402
Connections:
- net labels added: LED_1, LED_2
- wire segments 777 -> 787
Other:
- note added: "LED INDICATORS"
- note removed: "Locked_signal_led"

Commit message: Rework the layout of SDI input and output path
Parts:
- gave numbers to parts that had none: 4
Connections:
- net labels added: SDI_N, SDI_P, SDO_N, SDO_P
- net labels removed: SDI, SDO, ~SDI~, ~SDO~
Changed lines of the file:
@@
 	10650 6500 10650 6250
 Text Label 11700 5350 2    50   ~ 0
-SDI
+SDI_P
 Text Label 11700 5750 2    50   ~ 0
-~SDI~
+SDI_N
 Wire Wire Line
 	10650 5750 10650 5950
@@
 AUDIO_MASTER_CLK
 Text Label 2750 6100 0    50   ~ 0
-~SDO~
+SDO_N
 Text Label 2750 6000 0    50   ~ 0
-SDO
+SDO_P
 Wire Notes Line
 	16000 4900 13950 4900
@@
 $EndComp
 Text Label 1250 3550 0    50   ~ 0
-SDO
+SDO_P
 Text Label 1250 3650 0    50   ~ 0
-~SDO~
+SDO_N
 Wire Wire Line
 	2250 3550 1250 3550
@@
 $EndComp
 Text Label 5750 3400 0    50   ~ 0
-~SDI~
+SDI_N
 Text Label 5750 3300 0    50   ~ 0
-SDI
+SDI_P
 Wire Wire Line
 	6450 3400 5750 3400
@@
 LED_2
 $Comp
-L SDI-bridge:R_100R_0402 R?
+L SDI-bridge:R_100R_0402 R92
 U 1 1 5EDD71C4
 P 14750 6550
-F 0 "R?" H 14750 6650 60  0000 L CNN
+F 0 "R92" H 14750 6650 60  0000 L CNN
 F 1 "R_100R_0402" H 14750 6400 60  0001 C CNN
 F 2 "SDI-bridge-footprints:0402-res" H 14950 6750 60  0001 L CNN
@@
 $EndComp
 $Comp
-L SDI-bridge:LG_L29K-G2J1-24-Z D?
+L SDI-bridge:LG_L29K-G2J1-24-Z D3
 U 1 1 5EDD71CC
 P 15350 6550
-F 0 "D?" H 15350 6450 60  0000 R CNN
+F 0 "D3" H 15350 6450 60  0000 R CNN
 F 1 "LG_L29K-G2J1-24-Z" H 15650 6800 60  0000 R CNN
 F 2 "SDI-bridge-footprints:LED_0603" H 15550 6750 60  0001 L CNN
@@
 P 15850 6650
 AR Path="/5DD55102/5EDD71D5" Ref="#PWR?"  Part="1"
-AR Path="/5EDD71D5" Ref="#PWR?"  Part="1"
-F 0 "#PWR?" H 15850 6400 50  0001 C CNN
+AR Path="/5EDD71D5" Ref="#PWR0113"  Part="1"
+F 0 "#PWR0113" H 15850 6400 50  0001 C CNN
 F 1 "GNDA" H 15855 6477 50  0000 C CNN
 F 2 "" H 15850 6650 50  0001 C CNN
@@
 	14050 6550 14600 6550
 $Comp
-L SDI-bridge:R_100R_0402 R?
+L SDI-bridge:R_100R_0402 R93
 U 1 1 5EE8527F
 P 14750 7100
-F 0 "R?" H 14750 7200 60  0000 L CNN
+F 0 "R93" H 14750 7200 60  0000 L CNN
 F 1 "R_100R_0402" H 14750 6950 60  0001 C CNN
 F 2 "SDI-bridge-footprints:0402-res" H 14950 7300 60  0001 L CNN
@@
 $EndComp
 $Comp
-L SDI-bridge:LG_L29K-G2J1-24-Z D?
+L SDI-bridge:LG_L29K-G2J1-24-Z D4
 U 1 1 5EE85287
 P 15350 7100
-F 0 "D?" H 15350 7000 60  0000 R CNN
+F 0 "D4" H 15350 7000 60  0000 R CNN
 F 1 "LG_L29K-G2J1-24-Z" H 15650 7350 60  0000 R CNN
 F 2 "SDI-bridge-footprints:LED_0603" H 15550 7300 60  0001 L CNN
@@
 P 15850 7200
 AR Path="/5DD55102/5EE85290" Ref="#PWR?"  Part="1"
-AR Path="/5EE85290" Ref="#PWR?"  Part="1"
-F 0 "#PWR?" H 15850 6950 50  0001 C CNN
+AR Path="/5EE85290" Ref="#PWR0114"  Part="1"
+F 0 "#PWR0114" H 15850 6950 50  0001 C CNN
 F 1 "GNDA" H 15855 7027 50  0000 C CNN
 F 2 "" H 15850 7200 50  0001 C CNN

Commit message: Add several components to simplify the debugging process
-Add DIP switches for GS external configuration
-Make PCB a bit widther
-Move monting holes to the board sides
-Move power supply components
-Add Programming connectors
-Expose all audio pins at header
-Add GS reset button
-Add 2x user led and data error led
Parts:
- removed J4: MC-HVT1-S04-G, SDI-bridge-footprints:PinHeader_1x4_P1.27mm_Drill.7mm, symbol SDI-bridge:MC-HVT1-S04-G
- removed J6: MC-HVT1-S04-G, antmicro-footprints:PinHeader_1x4_P1.27mm_Drill.7mm, symbol antmicroRectangularConnectorsHeadersMalePins:MC-HVT1-S04-G
- removed R64, R65, R66, R68: R_2k37_0402, SDI-bridge-footprints:0402-res, symbol SDI-bridge:R_2k37_0402
- removed R75, R76, R77, R78, R79, R80, R81, R82, R83, R84, R85, R86, R87: R_0R_0402, SDI-bridge-footprints:0402-res, symbol SDI-bridge:R_0R_0402
- removed TP22, TP3, TP4, TP5: TP_SMD1MM, SDI-bridge-footprints:Testpoint_smd_1mm, symbol SDI-bridge:TP_SMD1MM
- added D5: LG_L29K-G2J1-24-Z, SDI-bridge-footprints:LED_0603, symbol SDI-bridge:LG_L29K-G2J1-24-Z
- added J4, J6: 2199SB-10G-301523, antmicro-footprints:PinHeader_2x05_P1.27mm_Vertical, symbol antmicroRectangularConnectorsHeadersMalePins:2199SB-10G-301523
- added R64: R_100R_0402, SDI-bridge-footprints:0402-res, symbol SDI-bridge:R_100R_0402
- added R65, R66, R68, R75, R76, R77, R78, R79, R80, R81, R82, R83: R_10k_0402, antmicro-footprints:0402-res, symbol antmicroResistors0402:R_10k_0402
- added R84, R85, R86, R87, R94: R_2k2_0402, antmicro-footprints:0402-res, symbol antmicroResistors0402:R_2k2_0402
- added R95: R_4k7_0402, SDI-bridge-footprints:0402-res, symbol SDI-bridge:R_4k7_0402
- added R96: R_30R_0402, antmicro-footprints:0402-res, symbol antmicroResistors0402:R_30R_0402
- added S1: B3U-1000P, antmicro-footprints:Switch_Tactile_SMD_B3U-1000P, symbol antmicroTactileSwitches:B3U-1000P
- added SW1, SW2: SW_DIP_x06, antmicro-footprints:SW_SPST_6_Slide_MCDHN-06F-T-V_P1.27mm, symbol antmicroSlideSwitches:SW_DIP_x06
Connections:
- net labels added: CRESET_B, MISO, MOSI, SPI_SCK(SDA), SPI_SS(SCL), USER_SCL, USER_SDA
- wire segments 787 -> 868
- no-connect marks 4 -> 5
Other:
- note added: "Conf DIP Switches"
- note added: "CrossLink programming connector"
- note added: "GS_I2C"
- note added: "RESET_Switch"
- note removed: "I2C exposed at goldpins"
- note removed: "Unused Audio chanels"

Commit message: Define release 1.0.0
Other:
- note added: "CrossLink"
- note removed: "Cross Link"
Changed lines of the file:
@@
 encoding utf-8
 Sheet 1 1
-Title ""
+Title "SDI Bridge"
 Date ""
-Rev ""
-Comp ""
-Comment1 ""
+Rev "1.1.0"
+Comp "Antmicro Ltd."
+Comment1 "Jakub Krzyska"
 Comment2 ""
 Comment3 ""
@@
 GS2971A
 Text Notes 16850 8000 0    118  ~ 24
-Cross Link
+CrossLink
 Text Notes 19300 5100 0    79   ~ 16
 I2C pull-ups

Commit message: Add OSHW logo and fix CS pin
There are following changes made:
-Disconnect CS pin from dip switch
-Replace one user led with user switch
-Remove leftovers form previous revision
-Update date and revision
Parts:
- removed D3: LG_L29K-G2J1-24-Z, SDI-bridge-footprints:LED_0603, symbol SDI-bridge:LG_L29K-G2J1-24-Z
- removed R92: R_100R_0402, SDI-bridge-footprints:0402-res, symbol SDI-bridge:R_100R_0402
- added N2: oshw_logo, antmicro-footprints:oshw-logo, symbol antmicroMechanicalParts:oshw_logo
Connections:
- net labels added: USER_LED, USER_SW
- net labels removed: LED_1, LED_2
- wire segments 868 -> 864
Changed lines of the file:
@@
 L SDI-bridge:antmicro_logo N1
 U 1 1 5FE7A74E
-P 1000 7150
-F 0 "N1" H 1214 7243 50  0000 L CNN
-F 1 "antmicro_logo" H 1214 7152 50  0000 L CNN
-F 2 "SDI-bridge-footprints:antmicro-logo_scaled_20mm" H 900 7400 50  0001 C CNN
-F 3 "" H 1000 7500 50  0001 C CNN
-	1    1000 7150
+P 800 7200
+F 0 "N1" H 1014 7293 50  0000 L CNN
+F 1 "antmicro_logo" H 1014 7202 50  0000 L CNN
+F 2 "SDI-bridge-footprints:antmicro-logo_scaled_20mm" H 700 7450 50  0001 C CNN
+F 3 "" H 800 7550 50  0001 C CNN
+	1    800  7200
 	1    0    0    -1
 $EndComp
@@
 Wire Wire Line
 	17000 13050 18000 13050
-Text Label 17000 13050 0    50   ~ 0
-LED_1
 Wire Wire Line
 	17000 13150 18000 13150
 Text Label 17000 13150 0    50   ~ 0
-LED_2
-$Comp
-L SDI-bridge:R_100R_0402 R92
-U 1 1 5EDD71C4
-P 12800 9600
-F 0 "R92" H 12800 9700 60  0000 L CNN
-F 1 "R_100R_0402" H 12800 9450 60  0001 C CNN
-F 2 "SDI-bridge-footprints:0402-res" H 13000 9800 60  0001 L CNN
-F 3 "" H 12800 9600 50  0001 C CNN
-F 4 "BOURNS" H 13000 10000 60  0001 L CNN "Manufacturer"
-F 5 "CR0402-FX-1000GLF" H 13000 9900 60  0001 L CNN "MPN"
-F 6 "100R" H 12700 9500 50  0000 L CNN "Val"
-	1    12800 9600
-	-1   0    0    -1
-$EndComp
-$Comp
-L SDI-bridge:LG_L29K-G2J1-24-Z D3
-U 1 1 5EDD71CC
-P 13400 9600
-F 0 "D3" H 13400 9500 60  0000 R CNN
-F 1 "LG_L29K-G2J1-24-Z" H 13700 9850 60  0000 R CNN
-F 2 "SDI-bridge-footprints:LED_0603" H 13600 9800 60  0001 L CNN
-F 3 "https://dammedia.osram.info/media/resource/hires/osram-dam-2493945/LG%20L29K.pdf" H 13600 9900 60  0001 L CNN
-F 4 "LG L29K-G2J1-24-Z" H 13600 10100 60  0001 L CNN "MPN"
-F 5 "OSRAM Opto Semiconductors Inc." H 13600 10700 60  0001 L CNN "Manufacturer"
-	1    13400 9600
-	1    0    0    1
-$EndComp
-Wire Wire Line
-	12950 9600 13200 9600
-Wire Wire Line
-	13900 9600 13900 9700
-Wire Wire Line
-	13500 9600 13900 9600
-Text Label 12100 9600 0    50   ~ 0
-LED_1
-Wire Wire Line
-	12100 9600 12650 9600
+USER_LED
 $Comp
 L SDI-bridge:R_100R_0402 R93
 U 1 1 5EE8527F
-P 12800 10150
-F 0 "R93" H 12800 10250 60  0000 L CNN
-F 1 "R_100R_0402" H 12800 10000 60  0001 C CNN
-F 2 "SDI-bridge-footprints:0402-res" H 13000 10350 60  0001 L CNN
-F 3 "" H 12800 10150 50  0001 C CNN
-F 4 "BOURNS" H 13000 10550 60  0001 L CNN "Manufacturer"
-F 5 "CR0402-FX-1000GLF" H 13000 10450 60  0001 L CNN "MPN"
-F 6 "100R" H 12700 10050 50  0000 L CNN "Val"
-	1    12800 10150
+P 12800 9650
+F 0 "R93" H 12800 9750 60  0000 L CNN
+F 1 "R_100R_0402" H 12800 9500 60  0001 C CNN
+F 2 "SDI-bridge-footprints:0402-res" H 13000 9850 60  0001 L CNN
+F 3 "" H 12800 9650 50  0001 C CNN
+F 4 "BOURNS" H 13000 10050 60  0001 L CNN "Manufacturer"
+F 5 "CR0402-FX-1000GLF" H 13000 9950 60  0001 L CNN "MPN"
+F 6 "100R" H 12700 9550 50  0000 L CNN "Val"
+	1    12800 9650
 	-1   0    0    -1
 $EndComp
@@
 L SDI-bridge:LG_L29K-G2J1-24-Z D4
 U 1 1 5EE85287
-P 13400 10150
-F 0 "D4" H 13400 10050 60  0000 R CNN
-F 1 "LG_L29K-G2J1-24-Z" H 13700 10400 60  0000 R CNN
-F 2 "SDI-bridge-footprints:LED_0603" H 13600 10350 60  0001 L CNN
-F 3 "https://dammedia.osram.info/media/resource/hires/osram-dam-2493945/LG%20L29K.pdf" H 13600 10450 60  0001 L CNN
-F 4 "LG L29K-G2J1-24-Z" H 13600 10650 60  0001 L CNN "MPN"
-F 5 "OSRAM Opto Semiconductors Inc." H 13600 11250 60  0001 L CNN "Manufacturer"
-	1    13400 10150
+P 13400 9650
+F 0 "D4" H 13400 9550 60  0000 R CNN
+F 1 "LG_L29K-G2J1-24-Z" H 13700 9900 60  0000 R CNN
+F 2 "SDI-bridge-footprints:LED_0603" H 13600 9850 60  0001 L CNN
+F 3 "https://dammedia.osram.info/media/resource/hires/osram-dam-2493945/LG%20L29K.pdf" H 13600 9950 60  0001 L CNN
+F 4 "LG L29K-G2J1-24-Z" H 13600 10150 60  0001 L CNN "MPN"
+F 5 "OSRAM Opto Semiconductors Inc." H 13600 10750 60  0001 L CNN "Manufacturer"
+	1    13400 9650
 	1    0    0    1
 $EndComp
 Wire Wire Line
-	12950 10150 13200 10150
+	12950 9650 13200 9650
 Wire Wire Line
-	13900 10150 13900 10250
+	13900 9650 13900 9750
 Wire Wire Line
-	13500 10150 13900 10150
-Text Label 12100 10150 0    50   ~ 0
-LED_2
+	13500 9650 13900 9650
+Text Label 12100 9650 0    50   ~ 0
+USER_LED
 Wire Wire Line
-	12100 10150 12650 10150
+	12100 9650 12650 9650
 Wire Notes Line
 	19100 650  19100 7450
@@
 L SDI-bridge:R_100R_0402 R64
 U 1 1 5FD0CB96
-P 12850 10750
-F 0 "R64" H 12850 10850 60  0000 L CNN
-F 1 "R_100R_0402" H 12850 10600 60  0001 C CNN
-F 2 "SDI-bridge-footprints:0402-res" H 13050 10950 60  0001 L CNN
-F 3 "" H 12850 10750 50  0001 C CNN
-F 4 "BOURNS" H 13050 11150 60  0001 L CNN "Manufacturer"
-F 5 "CR0402-FX-1000GLF" H 13050 11050 60  0001 L CNN "MPN"
-F 6 "100R" H 12750 10650 50  0000 L CNN "Val"
-	1    12850 10750
+P 12850 10250
+F 0 "R64" H 12850 10350 60  0000 L CNN
+F 1 "R_100R_0402" H 12850 10100 60  0001 C CNN
+F 2 "SDI-bridge-footprints:0402-res" H 13050 10450 60  0001 L CNN
+F 3 "" H 12850 10250 50  0001 C CNN
+F 4 "BOURNS" H 13050 10650 60  0001 L CNN "Manufacturer"
+F 5 "CR0402-FX-1000GLF" H 13050 10550 60  0001 L CNN "MPN"
+F 6 "100R" H 12750 10150 50  0000 L CNN "Val"
+	1    12850 10250
 	-1   0    0    -1
 $EndComp
@@
 L SDI-bridge:LG_L29K-G2J1-24-Z D5
 U 1 1 5FD0CB9E
-P 13450 10750
-F 0 "D5" H 13450 10650 60  0000 R CNN
-F 1 "LG_L29K-G2J1-24-Z" H 13750 11000 60  0000 R CNN
-F 2 "SDI-bridge-footprints:LED_0603" H 13650 10950 60  0001 L CNN
-F 3 "https://dammedia.osram.info/media/resource/hires/osram-dam-2493945/LG%20L29K.pdf" H 13650 11050 60  0001 L CNN
-F 4 "LG L29K-G2J1-24-Z" H 13650 11250 60  0001 L CNN "MPN"
-F 5 "OSRAM Opto Semiconductors Inc." H 13650 11850 60  0001 L CNN "Manufacturer"
-	1    13450 10750
+P 13450 10250
+F 0 "D5" H 13450 10150 60  0000 R CNN
+F 1 "LG_L29K-G2J1-24-Z" H 13750 10500 60  0000 R CNN
+F 2 "SDI-bridge-footprints:LED_0603" H 13650 10450 60  0001 L CNN
+F 3 "https://dammedia.osram.info/media/resource/hires/osram-dam-2493945/LG%20L29K.pdf" H 13650 10550 60  0001 L CNN
+F 4 "LG L29K-G2J1-24-Z" H 13650 10750 60  0001 L CNN "MPN"
+F 5 "OSRAM Opto Semiconductors Inc." H 13650 11350 60  0001 L CNN "Manufacturer"
+	1    13450 10250
 	1    0    0    1
 $EndComp
 Wire Wire Line
-	13000 10750 13250 10750
+	13000 10250 13250 10250
 Wire Wire Line
-	13900 10750 13900 10850
+	13900 10250 13900 10350
 Wire Wire Line
-	13550 10750 13900 10750
-Text Label 12150 10750 0    50   ~ 0
+	13550 10250 13900 10250
+Text Label 12150 10250 0    50   ~ 0
 DATA_ERRORb
 $Comp
@@
 	1    0    0    -1
 $EndComp
-Text Label 12150 13400 0    50   ~ 0
-~CS~_TMS
 Text Label 12150 14750 0    50   ~ 0
 STANDBY
@@
 	19900 4350 19900 4450
 Wire Wire Line
-	12150 10750 12700 10750
+	12150 10250 12700 10250
 Text Label 16950 9050 0    50   ~ 0
 CRESET_B
@@
 L SDI-bridge:GNDREF #PWR?
 U 1 1 5F3163ED
-P 13900 10850
+P 13900 10350
 AR Path="/5DD55102/5F3163ED" Ref="#PWR?"  Part="1"
-AR Path="/5F3163ED" Ref="#PWR?"  Part="1"
-F 0 "#PWR?" H 13900 10600 50  0001 C CNN
-F 1 "GNDREF" H 13905 10677 50  0000 C CNN
-F 2 "" H 13900 10850 50  0001 C CNN
-F 3 "" H 13900 10850 50  0001 C CNN
-	1    13900 10850
+AR Path="/5F3163ED" Ref="#PWR0106"  Part="1"
+F 0 "#PWR0106" H 13900 10100 50  0001 C CNN
+F 1 "GNDREF" H 13905 10177 50  0000 C CNN
+F 2 "" H 13900 10350 50  0001 C CNN
+F 3 "" H 13900 10350 50  0001 C CNN
+	1    13900 10350
 	1    0    0    -1
 $EndComp
@@
 L SDI-bridge:GNDREF #PWR?
 U 1 1 5F3E1049
-P 13900 10250
+P 13900 9750
 AR Path="/5DD55102/5F3E1049" Ref="#PWR?"  Part="1"
-AR Path="/5F3E1049" Ref="#PWR?"  Part="1"
-F 0 "#PWR?" H 13900 10000 50  0001 C CNN
-F 1 "GNDREF" H 13905 10077 50  0000 C CNN
-F 2 "" H 13900 10250 50  0001 C CNN
-F 3 "" H 13900 10250 50  0001 C CNN
-	1    13900 10250
-	1    0    0    -1
-$EndComp
-$Comp
-L SDI-bridge:GNDREF #PWR?
-U 1 1 5F4ABD7F
-P 13900 9700
-AR Path="/5DD55102/5F4ABD7F" Ref="#PWR?"  Part="1"
-AR Path="/5F4ABD7F" Ref="#PWR?"  Part="1"
-F 0 "#PWR?" H 13900 9450 50  0001 C CNN
-F 1 "GNDREF" H 13905 9527 50  0000 C CNN
-F 2 "" H 13900 9700 50  0001 C CNN
-F 3 "" H 13900 9700 50  0001 C CNN
-	1    13900 9700
+AR Path="/5F3E1049" Ref="#PWR0113"  Part="1"
+F 0 "#PWR0113" H 13900 9500 50  0001 C CNN
+F 1 "GNDREF" H 13905 9577 50  0000 C CNN
+F 2 "" H 13900 9750 50  0001 C CNN
+F 3 "" H 13900 9750 50  0001 C CNN
+	1    13900 9750
 	1    0    0    -1
 $EndComp
@@
 P 13900 9200
 AR Path="/5DD55102/5F576A90" Ref="#PWR?"  Part="1"
-AR Path="/5F576A90" Ref="#PWR?"  Part="1"
-F 0 "#PWR?" H 13900 8950 50  0001 C CNN
+AR Path="/5F576A90" Ref="#PWR0116"  Part="1"
+F 0 "#PWR0116" H 13900 8950 50  0001 C CNN
 F 1 "GNDREF" H 13905 9027 50  0000 C CNN
 F 2 "" H 13900 9200 50  0001 C CNN
@@
 P 13900 8450
 AR Path="/5DD55102/5F6417DF" Ref="#PWR?"  Part="1"
-AR Path="/5F6417DF" Ref="#PWR?"  Part="1"
-F 0 "#PWR?" H 13900 8200 50  0001 C CNN
+AR Path="/5F6417DF" Ref="#PWR0119"  Part="1"
+F 0 "#PWR0119" H 13900 8200 50  0001 C CNN
 F 1 "GNDREF" H 13905 8277 50  0000 C CNN
 F 2 "" H 13900 8450 50  0001 C CNN
@@
 Wire Notes Line
 	11850 11700 15350 11700
+$Comp
+L antmicroMechanicalParts:oshw_logo N2
+U 1 1 5ED060A3
+P 1800 7100
+F 0 "N2" H 1994 7103 50  0000 L CNN
+F 1 "oshw_logo" H 1994 7012 50  0000 L CNN
+F 2 "antmicro-footprints:oshw-logo" H 1820 6860 50  0001 C CNN
+F 3 "" H 1800 7100 50  0001 C CNN
+	1    1800 7100
+	1    0    0    -1
+$EndComp
+Text Label 12150 13400 0    50   ~ 0
+USER_SW
+Text Label 17000 13050 0    50   ~ 0
+USER_SW
 Wire Bus Line
 	16900 10650 16900 11550

Commit message: Library updates
Other:
- note added: "Configuration DIP Switches"
- note added: "CrossLink MIPI transmitter"
- note added: "Logotypes"
- note added: "Programming interace"
- note added: "Pull-up resistors"
- note added: "RESET"
- note added: "SDI deserializer"
- note added: "SDI input"
- note added: "SDI output"
- note removed: "Conf DIP Switches"
- note removed: "CrossLink"
- note removed: "CrossLink programming connector"
- note removed: "GS2971A"
- note removed: "I2C pull-ups"
- note removed: "Logo"
- note removed: "RESET_Switch"
- note removed: "SDI input signal"
- note removed: "SDO\n"
Changed lines of the file:
@@
 encoding utf-8
 Sheet 1 1
-Title "SDI Bridge"
+Title "SDI-MIPI Bridge"
 Date ""
 Rev "1.1.0"
-Comp "Antmicro Ltd."
-Comment1 "Jakub Krzyska"
-Comment2 ""
+Comp ""
+Comment1 "www.antmicro.com"
+Comment2 "Antmicro Ltd."
 Comment3 ""
 Comment4 ""
@@
 	10500 6500 10650 6500
 Text Notes 8900 4700 0    79   ~ 16
-SDI input signal
+SDI input
 Wire Wire Line
 	9150 5550 9150 5750
@@
 	12800 6550 12800 6700
 Text Notes 12450 4700 0    59   ~ 12
-Place close to GS2971A
+Filtering
 Wire Wire Line
 	15050 4450 15900 4450
@@
 	450  4450 13950 4450
 Wire Notes Line
-	2550 4750 2550 7450
+	2550 4450 2550 7450
 Wire Wire Line
 	3950 3550 3550 3550
@@
 	11800 4450 11800 16050
 Text Notes 500  6950 0    79   ~ 16
-Logo
+Logotypes
 Wire Wire Line
 	3200 6100 4050 6100
@@
 AUDIO_OUTPUT_CH7_8
 Text Notes 2750 4650 0    79   ~ 16
-SDO\n
+SDI output
 Wire Wire Line
 	3500 6200 4050 6200
@@
 Place close to GS2971A
 Text Notes 900  950  0    118  ~ 24
-GS2971A
+SDI deserializer
 Text Notes 16850 8000 0    118  ~ 24
-CrossLink
+CrossLink MIPI transmitter
 Text Notes 19300 5100 0    79   ~ 16
-I2C pull-ups
+Pull-up resistors
 Wire Wire Line
 	9900 13700 10300 13700
@@
 	17950 9650 18000 9650
 Text Notes 500  4650 0    79   ~ 16
-CrossLink programming connector
+Programming interace
 Text Notes 14050 5450 0    79   ~ 16
-RESET_Switch
+RESET
 $Comp
 L SDI-bridge:GNDREF #PWR?
@@
 $EndComp
 Text Notes 12100 12450 0    79   ~ 16
-Conf DIP Switches
+Configuration DIP Switches
 Wire Notes Line
 	15350 16050 15350 7450
