File: sdi-mipi-bridge.sch (KiCad schematic (older format))
At the start: 202 parts, among them J1 031-70526-21, J2 031-70526-21, J3 WE_68715014522_ONE-SIDE, J4 2199SB-10G-301523, J5 MC-HVT1-S04-G, J6 2199SB-10G-301523, SW1 SW_DIP_x06, SW2 SW_DIP_x06, U1 MAX8902B, U2 GS2971A, U3 GS2988, U4 CrossLink_LIF-MD6000-6JMG80I, U5 SC18IS602BIPW, Y1 ABM7_27.000MH_D2Y_T

Commit message: Fixed 3V3 reference
Connections:
- net labels added: +3V3
Changed lines of the file:
@@
 Text Label 17000 13050 0    50   ~ 0
 USER_SW
-Wire Bus Line
-	16900 10650 16900 11550
-Wire Bus Line
-	4850 2850 4850 3750
 $Comp
-L power:+3.3V #PWR?
+L sdi-mipi-bridge:+3V3 #PWR?
 U 1 1 5F0AA363
 P 5900 14150
@@
 $EndComp
 $Comp
-L power:+3.3V #PWR?
+L sdi-mipi-bridge:+3V3 #PWR?
 U 1 1 5F0AF54D
 P 5450 11950
@@
 $EndComp
 $Comp
-L power:+3.3V #PWR?
+L sdi-mipi-bridge:+3V3 #PWR?
 U 1 1 5F0B8283
 P 8850 8300
@@
 $EndComp
 $Comp
-L power:+3.3V #PWR?
-U 1 1 5F0BBC17
-P 5450 8600
-F 0 "#PWR?" H 5450 8450 50  0001 C CNN
-F 1 "+3.3V" H 5465 8773 50  0000 C CNN
-F 2 "" H 5450 8600 50  0001 C CNN
-F 3 "" H 5450 8600 50  0001 C CNN
-	1    5450 8600
-	1    0    0    -1
-$EndComp
-$Comp
-L power:+3.3V #PWR?
+L sdi-mipi-bridge:+3V3 #PWR?
 U 1 1 5F0C4337
 P 8700 14850
@@
 $EndComp
 $Comp
-L power:+3.3V #PWR?
+L sdi-mipi-bridge:+3V3 #PWR?
 U 1 1 5F0CE737
 P 1000 8900
@@
 $EndComp
 $Comp
-L power:+3.3V #PWR?
+L sdi-mipi-bridge:+3V3 #PWR?
 U 1 1 5F0D19F3
 P 1900 5900
@@
 $EndComp
 $Comp
-L power:+3.3V #PWR?
+L sdi-mipi-bridge:+3V3 #PWR?
 U 1 1 5F0D73D2
 P 650 4900
@@
 $EndComp
 $Comp
-L power:+3.3V #PWR?
+L sdi-mipi-bridge:+3V3 #PWR?
 U 1 1 5F0E97F8
 P 20200 8400
@@
 $EndComp
 $Comp
-L power:+3.3V #PWR?
+L sdi-mipi-bridge:+3V3 #PWR?
 U 1 1 5F0F58E5
 P 21400 5250
@@
 $EndComp
 $Comp
-L power:+3.3V #PWR?
+L sdi-mipi-bridge:+3V3 #PWR?
 U 1 1 5F0FDF23
 P 22650 1600
@@
 $EndComp
 $Comp
-L power:+3.3V #PWR?
+L sdi-mipi-bridge:+3V3 #PWR?
 U 1 1 5F0FE78D
 P 19350 1200
@@
 $EndComp
 $Comp
-L power:+3.3V #PWR?
+L sdi-mipi-bridge:+3V3 #PWR?
 U 1 1 5F104E29
 P 17750 5850
@@
 	1    0    0    -1
 $EndComp
+Wire Bus Line
+	16900 10650 16900 11550
+Wire Bus Line
+	4850 2850 4850 3750
+$Comp
+L sdi-mipi-bridge:+3V3 #PWR?
+U 1 1 5F1F5CC8
+P 5450 8600
+F 0 "#PWR?" H 5450 8450 50  0001 C CNN
+F 1 "+3V3" H 5465 8773 50  0000 C CNN
+F 2 "" H 5450 8600 50  0001 C CNN
+F 3 "" H 5450 8600 50  0001 C CNN
+	1    5450 8600
+	1    0    0    -1
+$EndComp

Commit message: Added missing MPNs
Parts:
- U3: MPN GS2988-INTE3 -> GS2988-INE3
- U4: Manufacturer (none) -> Lattice Semiconductor
- U5: MPN (none) -> SC18IS602BIPW; Manufacturer (none) -> NXP
Changed lines of the file:
@@
 EESchema Schematic File Version 4
+LIBS:sdi-mipi-bridge-cache
 EELAYER 30 0
 EELAYER END
@@
 F 4 "LIF-MD6000-6JMG80I" H 18600 9625 50  0000 C CNN "MPN"
 F 5 "Lattice Semiconductor" H 18600 9725 50  0000 C CNN "Manufacurer"
+F 6 "Lattice Semiconductor" H 18000 9250 50  0001 C CNN "Manufacturer"
 	1    18000 9250
 	1    0    0    -1
@@
 F 2 "sdi-mipi-bridge-footprints:QFN-16_EP_4x4_Pitch0.65mm" H 4050 5950 60  0001 R CNN
 F 3 "https://semtech.my.salesforce.com/sfc/p/E0000000JelG/a/44000000MDIY/URmNPYk6YrvngFjCh2n.ZRVsjLb90QOH1YLezdH9vhM" H 4050 5750 60  0001 R CNN
-F 4 "GS2988-INTE3" H 5150 5100 50  0000 C CNN "MPN"
+F 4 "GS2988-INE3" H 5150 5100 50  0000 C CNN "MPN"
 F 5 "Semtech" H 5025 5200 50  0000 C CNN "Manufacturer"
 	1    3900 5900
@@
 F 1 "SC18IS602BIPW" H 20800 800 60  0000 C CNN
 F 2 "sdi-mipi-bridge-footprints:SC18IS602B" H 20450 1750 60  0001 L CNN
-F 3 "" H 20450 1550 60  0001 L CNN
+F 3 "https://www.nxp.com/docs/en/data-sheet/SC18IS602B.pdf" H 20450 1550 60  0001 L CNN
+F 4 "SC18IS602BIPW" H 20250 1700 50  0001 C CNN "MPN"
+F 5 "NXP" H 20250 1700 50  0001 C CNN "Manufacturer"
 	1    20250 1700
 	1    0    0    -1
@@
 U 1 1 656F6957
 P 13050 15150
-F 0 "R77" V 12900 15000 60  0000 L CNN
+F 0 "R77" H 13350 15125 60  0000 L CNN
 F 1 "R_10k_0402" H 13050 15000 60  0001 C CNN
 F 2 "sdi-mipi-bridge-footprints:0402-res" H 13250 15350 60  0001 L CNN
@@
 U 1 1 67587E9D
 P 12900 15150
-F 0 "R75" V 12750 15000 60  0000 L CNN
+F 0 "R75" H 13200 15125 60  0000 L CNN
 F 1 "R_10k_0402" H 12900 15000 60  0001 C CNN
 F 2 "sdi-mipi-bridge-footprints:0402-res" H 13100 15350 60  0001 L CNN
@@
 U 1 1 675883BE
 P 13500 13150
-F 0 "R66" V 13350 13000 60  0000 L CNN
+F 0 "R66" H 13050 13100 60  0000 L CNN
 F 1 "R_10k_0402" H 13500 13000 60  0001 C CNN
 F 2 "sdi-mipi-bridge-footprints:0402-res" H 13700 13350 60  0001 L CNN
@@
 U 1 1 6758887B
 P 13200 15150
-F 0 "R79" V 13050 15000 60  0000 L CNN
+F 0 "R79" H 13500 15100 60  0000 L CNN
 F 1 "R_10k_0402" H 13200 15000 60  0001 C CNN
 F 2 "sdi-mipi-bridge-footprints:0402-res" H 13400 15350 60  0001 L CNN
@@
 U 1 1 67588C94
 P 13350 15150
-F 0 "R81" V 13200 15000 60  0000 L CNN
+F 0 "R81" H 13650 15100 60  0000 L CNN
 F 1 "R_10k_0402" H 13350 15000 60  0001 C CNN
 F 2 "sdi-mipi-bridge-footprints:0402-res" H 13550 15350 60  0001 L CNN
@@
 U 1 1 675891E1
 P 13500 15150
-F 0 "R83" V 13350 15000 60  0000 L CNN
+F 0 "R83" H 13800 15100 60  0000 L CNN
 F 1 "R_10k_0402" H 13500 15000 60  0001 C CNN
 F 2 "sdi-mipi-bridge-footprints:0402-res" H 13700 15350 60  0001 L CNN
@@
 U 1 1 67B0EE6A
 P 13050 13150
-F 0 "R76" V 12900 13000 60  0000 L CNN
+F 0 "R76" H 12600 13100 60  0000 L CNN
 F 1 "R_10k_0402" H 13050 13000 60  0001 C CNN
 F 2 "sdi-mipi-bridge-footprints:0402-res" H 13250 13350 60  0001 L CNN
@@
 U 1 1 67B0EE73
 P 12900 13150
-F 0 "R68" V 12750 13000 60  0000 L CNN
+F 0 "R68" H 12450 13125 60  0000 L CNN
 F 1 "R_10k_0402" H 12900 13000 60  0001 C CNN
 F 2 "sdi-mipi-bridge-footprints:0402-res" H 13100 13350 60  0001 L CNN
@@
 U 1 1 67B0EE7C
 P 13650 15150
-F 0 "R65" V 13500 15000 60  0000 L CNN
+F 0 "R65" H 13950 15100 60  0000 L CNN
 F 1 "R_10k_0402" H 13650 15000 60  0001 C CNN
 F 2 "sdi-mipi-bridge-footprints:0402-res" H 13850 15350 60  0001 L CNN
@@
 U 1 1 67B0EE85
 P 13200 13150
-F 0 "R78" V 13050 13000 60  0000 L CNN
+F 0 "R78" H 12750 13100 60  0000 L CNN
 F 1 "R_10k_0402" H 13200 13000 60  0001 C CNN
 F 2 "sdi-mipi-bridge-footprints:0402-res" H 13400 13350 60  0001 L CNN
@@
 U 1 1 67B0EE8E
 P 13350 13150
-F 0 "R80" V 13200 13000 60  0000 L CNN
+F 0 "R80" H 12900 13100 60  0000 L CNN
 F 1 "R_10k_0402" H 13350 13000 60  0001 C CNN
 F 2 "sdi-mipi-bridge-footprints:0402-res" H 13550 13350 60  0001 L CNN
@@
 U 1 1 67B0EE97
 P 13650 13150
-F 0 "R82" V 13500 13000 60  0000 L CNN
+F 0 "R82" H 13200 13100 60  0000 L CNN
 F 1 "R_10k_0402" H 13650 13000 60  0001 C CNN
 F 2 "sdi-mipi-bridge-footprints:0402-res" H 13850 13350 60  0001 L CNN
@@
 USER_SW
 $Comp
-L sdi-mipi-bridge:+3V3 #PWR?
+L sdi-mipi-bridge:+3V3 #PWR0114
 U 1 1 5F0AA363
 P 5900 14150
-F 0 "#PWR?" H 5900 14000 50  0001 C CNN
+F 0 "#PWR0114" H 5900 14000 50  0001 C CNN
 F 1 "+3.3V" H 5915 14323 50  0000 C CNN
 F 2 "" H 5900 14150 50  0001 C CNN
@@
 $EndComp
 $Comp
-L sdi-mipi-bridge:+3V3 #PWR?
+L sdi-mipi-bridge:+3V3 #PWR0120
 U 1 1 5F0AF54D
 P 5450 11950
-F 0 "#PWR?" H 5450 11800 50  0001 C CNN
+F 0 "#PWR0120" H 5450 11800 50  0001 C CNN
 F 1 "+3.3V" H 5465 12123 50  0000 C CNN
 F 2 "" H 5450 11950 50  0001 C CNN
@@
 $EndComp
 $Comp
-L sdi-mipi-bridge:+3V3 #PWR?
+L sdi-mipi-bridge:+3V3 #PWR0121
 U 1 1 5F0B8283
 P 8850 8300
-F 0 "#PWR?" H 8850 8150 50  0001 C CNN
+F 0 "#PWR0121" H 8850 8150 50  0001 C CNN
 F 1 "+3.3V" H 8865 8473 50  0000 C CNN
 F 2 "" H 8850 8300 50  0001 C CNN
@@
 $EndComp
 $Comp
-L sdi-mipi-bridge:+3V3 #PWR?
+L sdi-mipi-bridge:+3V3 #PWR0122
 U 1 1 5F0C4337
 P 8700 14850
-F 0 "#PWR?" H 8700 14700 50  0001 C CNN
+F 0 "#PWR0122" H 8700 14700 50  0001 C CNN
 F 1 "+3.3V" H 8715 15023 50  0000 C CNN
 F 2 "" H 8700 14850 50  0001 C CNN
@@
 $EndComp
 $Comp
-L sdi-mipi-bridge:+3V3 #PWR?
+L sdi-mipi-bridge:+3V3 #PWR0123
 U 1 1 5F0CE737
 P 1000 8900
-F 0 "#PWR?" H 1000 8750 50  0001 C CNN
+F 0 "#PWR0123" H 1000 8750 50  0001 C CNN
 F 1 "+3.3V" H 1015 9073 50  0000 C CNN
 F 2 "" H 1000 8900 50  0001 C CNN
@@
 $EndComp
 $Comp
-L sdi-mipi-bridge:+3V3 #PWR?
+L sdi-mipi-bridge:+3V3 #PWR0124
 U 1 1 5F0D19F3
 P 1900 5900
-F 0 "#PWR?" H 1900 5750 50  0001 C CNN
+F 0 "#PWR0124" H 1900 5750 50  0001 C CNN
 F 1 "+3.3V" H 1915 6073 50  0000 C CNN
 F 2 "" H 1900 5900 50  0001 C CNN
@@
 $EndComp
 $Comp
-L sdi-mipi-bridge:+3V3 #PWR?
+L sdi-mipi-bridge:+3V3 #PWR0125
 U 1 1 5F0D73D2
 P 650 4900
-F 0 "#PWR?" H 650 4750 50  0001 C CNN
+F 0 "#PWR0125" H 650 4750 50  0001 C CNN
 F 1 "+3.3V" H 665 5073 50  0000 C CNN
 F 2 "" H 650 4900 50  0001 C CNN
@@
 $EndComp
 $Comp
-L sdi-mipi-bridge:+3V3 #PWR?
+L sdi-mipi-bridge:+3V3 #PWR0126
 U 1 1 5F0E97F8
 P 20200 8400
-F 0 "#PWR?" H 20200 8250 50  0001 C CNN
+F 0 "#PWR0126" H 20200 8250 50  0001 C CNN
 F 1 "+3.3V" H 20215 8573 50  0000 C CNN
 F 2 "" H 20200 8400 50  0001 C CNN
@@
 $EndComp
 $Comp
-L sdi-mipi-bridge:+3V3 #PWR?
+L sdi-mipi-bridge:+3V3 #PWR0127
 U 1 1 5F0F58E5
 P 21400 5250
-F 0 "#PWR?" H 21400 5100 50  0001 C CNN
+F 0 "#PWR0127" H 21400 5100 50  0001 C CNN
 F 1 "+3.3V" H 21415 5423 50  0000 C CNN
 F 2 "" H 21400 5250 50  0001 C CNN
@@
 $EndComp
 $Comp
-L sdi-mipi-bridge:+3V3 #PWR?
+L sdi-mipi-bridge:+3V3 #PWR0128
 U 1 1 5F0FDF23
 P 22650 1600
-F 0 "#PWR?" H 22650 1450 50  0001 C CNN
+F 0 "#PWR0128" H 22650 1450 50  0001 C CNN
 F 1 "+3.3V" H 22665 1773 50  0000 C CNN
 F 2 "" H 22650 1600 50  0001 C CNN
@@
 $EndComp
 $Comp
-L sdi-mipi-bridge:+3V3 #PWR?
+L sdi-mipi-bridge:+3V3 #PWR0129
 U 1 1 5F0FE78D
 P 19350 1200
-F 0 "#PWR?" H 19350 1050 50  0001 C CNN
+F 0 "#PWR0129" H 19350 1050 50  0001 C CNN
 F 1 "+3.3V" H 19365 1373 50  0000 C CNN
 F 2 "" H 19350 1200 50  0001 C CNN
@@
 $EndComp
 $Comp
-L sdi-mipi-bridge:+3V3 #PWR?
+L sdi-mipi-bridge:+3V3 #PWR0130
 U 1 1 5F104E29
 P 17750 5850
-F 0 "#PWR?" H 17750 5700 50  0001 C CNN
+F 0 "#PWR0130" H 17750 5700 50  0001 C CNN
 F 1 "+3.3V" H 17765 6023 50  0000 C CNN
 F 2 "" H 17750 5850 50  0001 C CNN
@@
 	1    0    0    -1
 $EndComp
-Wire Bus Line
-	16900 10650 16900 11550
-Wire Bus Line
-	4850 2850 4850 3750
 $Comp
-L sdi-mipi-bridge:+3V3 #PWR?
+L sdi-mipi-bridge:+3V3 #PWR0131
 U 1 1 5F1F5CC8
 P 5450 8600
-F 0 "#PWR?" H 5450 8450 50  0001 C CNN
+F 0 "#PWR0131" H 5450 8450 50  0001 C CNN
 F 1 "+3V3" H 5465 8773 50  0000 C CNN
 F 2 "" H 5450 8600 50  0001 C CNN
@@
 	1    0    0    -1
 $EndComp
+Wire Bus Line
+	16900 10650 16900 11550
+Wire Bus Line
+	4850 2850 4850 3750
 $EndSCHEMATC

Commit message: Changed MFG and MPN for some parts to ease sourcing
Parts:
- C27: MPN MC0402B562K160CT -> C0402C562K3RACTU; Manufacturer Multicomp -> Kemet
- C38: MPN C1005X5R1A225K050BC -> C0402C225K9PACTU; Manufacturer TDK -> Kemet
- C63: MPN MC0402X473K160CT -> CGA2B2X7R1C473K050BA; Manufacturer MULTICOMP -> TDK
- FB1, FB2, FB3: value BLM18PG121SN1D -> BLM18PG121SH1D; MPN BLM18PG121SN1D -> BLM18PG121SH1D
- J4, J6: value 2199SB-10G-301523 -> GRPB052VWVN-RC; MPN 2199SB-10G-301523 -> GRPB052VWVN-RC; Manufacturer MULTICOMP PRO -> Sullins
- J5: value MC-HVT1-S04-G -> GRPB041VWVN-RC; MPN MC-HVT1-S04-G -> GRPB041VWVN-RC; Manufacturer Multicomp -> Sullins
- R17, R18, R19, R20, R27, R28: MPN MCWR06X75R0FTL -> RC0603FR-0775RL; Manufacturer MULTICOMP -> Yageo
- R29: MPN MCWR04X37R4FTL -> RC0402FR-0737R4L; Manufacturer Multicomp -> Yageo
- R30: MPN MC00625W04021105R -> RC0402FR-07105RL; Manufacturer Multicomp -> Yageo
- R5, R6: MPN CRCW0402120KFKED -> RC0402FR-07120KL; Manufacturer VISHAY -> Yageo
- SW1, SW2: MPN MCDHN-06F-T-V -> 97C06SRT; Manufacturer MULTICOMP PRO -> Grayhill
Changed lines of the file:
@@
 EESchema Schematic File Version 4
-LIBS:sdi-mipi-bridge-cache
 EELAYER 30 0
 EELAYER END
@@
 F 2 "sdi-mipi-bridge-footprints:0603-res" H 10500 6300 60  0001 L CNN
 F 3 "" H 10300 6100 50  0001 C CNN
-F 4 "MULTICOMP" H 10500 6500 60  0001 L CNN "Manufacturer"
-F 5 "MCWR06X75R0FTL" H 10500 6400 60  0001 L CNN "MPN"
+F 4 "Yageo" H 10500 6500 60  0001 L CNN "Manufacturer"
+F 5 "RC0603FR-0775RL" H 10500 6400 60  0001 L CNN "MPN"
 F 6 "75R" V 10450 6150 50  0000 L CNN "Val"
 	1    10300 6100
@@
 F 2 "sdi-mipi-bridge-footprints:0603-res" H 10050 5550 60  0001 L CNN
 F 3 "" H 9850 5350 50  0001 C CNN
-F 4 "MULTICOMP" H 10050 5750 60  0001 L CNN "Manufacturer"
-F 5 "MCWR06X75R0FTL" H 10050 5650 60  0001 L CNN "MPN"
+F 4 "Yageo" H 10050 5750 60  0001 L CNN "Manufacturer"
+F 5 "RC0603FR-0775RL" H 10050 5650 60  0001 L CNN "MPN"
 F 6 "75R" H 9750 5450 50  0000 L CNN "Val"
 	1    9850 5350
@@
 F 2 "sdi-mipi-bridge-footprints:0402-res" H 10850 6300 60  0001 L CNN
 F 3 "" H 10650 6100 50  0001 C CNN
-F 4 "Multicomp" H 10850 6500 60  0001 L CNN "Manufacturer"
-F 5 "MCWR04X37R4FTL" H 10850 6400 60  0001 L CNN "MPN"
+F 4 "Yageo" H 10850 6500 60  0001 L CNN "Manufacturer"
+F 5 "RC0402FR-0737R4L" H 10850 6400 60  0001 L CNN "MPN"
 F 6 "37R4" V 10800 6150 50  0000 L CNN "Val"
 	1    10650 6100
@@
 F 2 "sdi-mipi-bridge-footprints:0402-res" H 13000 5850 60  0001 L CNN
 F 3 "" H 12800 5650 50  0001 C CNN
-F 4 "Multicomp" H 13000 6050 60  0001 L CNN "Manufacturer"
-F 5 "MC00625W04021105R" H 13000 5950 60  0001 L CNN "MPN"
+F 4 "Yageo" H 13000 6050 60  0001 L CNN "Manufacturer"
+F 5 "RC0402FR-07105RL" H 13000 5950 60  0001 L CNN "MPN"
 F 6 "105R" V 12950 5700 50  0000 L CNN "Val"
 	1    12800 5650
@@
 F 2 "sdi-mipi-bridge-footprints:0402-cap" H 14850 3950 60  0001 L CNN
 F 3 "" H 14650 3750 50  0001 C CNN
-F 4 "MULTICOMP" H 14850 4150 60  0001 L CNN "Manufacturer"
-F 5 "MC0402X473K160CT" H 14850 4050 60  0001 L CNN "MPN"
+F 4 "TDK" H 14850 4150 60  0001 L CNN "Manufacturer"
+F 5 "CGA2B2X7R1C473K050BA" H 14850 4050 60  0001 L CNN "MPN"
 F 6 "47n" V 14600 3550 50  0000 L CNN "Val"
 	1    14650 3750
@@
 F 2 "sdi-mipi-bridge-footprints:0603-res" H 6600 6850 60  0001 L CNN
 F 3 "" H 6400 6650 50  0001 C CNN
-F 4 "MULTICOMP" H 6600 7050 60  0001 L CNN "Manufacturer"
-F 5 "MCWR06X75R0FTL" H 6600 6950 60  0001 L CNN "MPN"
+F 4 "Yageo" H 6600 7050 60  0001 L CNN "Manufacturer"
+F 5 "RC0603FR-0775RL" H 6600 6950 60  0001 L CNN "MPN"
 F 6 "75R" H 6550 6700 50  0000 L CNN "Val"
 	1    6400 6650
@@
 F 2 "sdi-mipi-bridge-footprints:0603-res" H 6600 5450 60  0001 L CNN
 F 3 "" H 6400 5250 50  0001 C CNN
-F 4 "MULTICOMP" H 6600 5650 60  0001 L CNN "Manufacturer"
-F 5 "MCWR06X75R0FTL" H 6600 5550 60  0001 L CNN "MPN"
+F 4 "Yageo" H 6600 5650 60  0001 L CNN "Manufacturer"
+F 5 "RC0603FR-0775RL" H 6600 5550 60  0001 L CNN "MPN"
 F 6 "75R" H 6550 5300 50  0000 L CNN "Val"
 	1    6400 5250
@@
 P 8850 10250
 F 0 "FB2" H 8850 10537 60  0000 C CNN
-F 1 "BLM18PG121SN1D" H 8850 10431 60  0000 C CNN
+F 1 "BLM18PG121SH1D" H 8850 10431 60  0000 C CNN
 F 2 "sdi-mipi-bridge-footprints:0603-res" H 9050 10450 60  0001 L CNN
 F 3 "https://www.murata.com/en-us/products/productdata/8796738650142/ENFA0003.pdf" H 9050 10550 60  0001 L CNN
-F 4 "BLM18PG121SN1D" H 9050 10750 60  0001 L CNN "MPN"
+F 4 "BLM18PG121SH1D" H 9050 10750 60  0001 L CNN "MPN"
 F 5 "Murata Electronics North America" H 9050 11350 60  0001 L CNN "Manufacturer"
 	1    8850 10250
@@
 P 8850 8550
 F 0 "FB1" H 8850 8837 60  0000 C CNN
-F 1 "BLM18PG121SN1D" H 8850 8731 60  0000 C CNN
+F 1 "BLM18PG121SH1D" H 8850 8731 60  0000 C CNN
 F 2 "sdi-mipi-bridge-footprints:0603-res" H 9050 8750 60  0001 L CNN
 F 3 "https://www.murata.com/en-us/products/productdata/8796738650142/ENFA0003.pdf" H 9050 8850 60  0001 L CNN
-F 4 "BLM18PG121SN1D" H 9050 9050 60  0001 L CNN "MPN"
+F 4 "BLM18PG121SH1D" H 9050 9050 60  0001 L CNN "MPN"
 F 5 "Murata Electronics North America" H 9050 9650 60  0001 L CNN "Manufacturer"
 	1    8850 8550
@@
 P 9350 13700
 F 0 "FB3" H 9350 13987 60  0000 C CNN
-F 1 "BLM18PG121SN1D" H 9350 13881 60  0000 C CNN
+F 1 "BLM18PG121SH1D" H 9350 13881 60  0000 C CNN
 F 2 "sdi-mipi-bridge-footprints:0603-res" H 9550 13900 60  0001 L CNN
 F 3 "https://www.murata.com/en-us/products/productdata/8796738650142/ENFA0003.pdf" H 9550 14000 60  0001 L CNN
-F 4 "BLM18PG121SN1D" H 9550 14200 60  0001 L CNN "MPN"
+F 4 "BLM18PG121SH1D" H 9550 14200 60  0001 L CNN "MPN"
 F 5 "Murata Electronics North America" H 9550 14800 60  0001 L CNN "Manufacturer"
 	1    9350 13700
@@
 F 2 "sdi-mipi-bridge-footprints:0402-cap" H 9050 11050 60  0001 L CNN
 F 3 "" H 8850 10850 50  0001 C CNN
-F 4 "TDK" H 9050 11250 60  0001 L CNN "Manufacturer"
-F 5 "C1005X5R1A225K050BC" H 9050 11150 60  0001 L CNN "MPN"
+F 4 "Kemet" H 9050 11250 60  0001 L CNN "Manufacturer"
+F 5 "C0402C225K9PACTU" H 9050 11150 60  0001 L CNN "MPN"
 F 6 "2u2" H 8900 10750 50  0000 L CNN "Val"
 	1    8850 10850
@@
 F 2 "sdi-mipi-bridge-footprints:0402-res" H 6600 5850 60  0001 L CNN
 F 3 "" H 6400 5650 50  0001 C CNN
-F 4 "Multicomp" H 6600 6050 60  0001 L CNN "Manufacturer"
-F 5 "MC0402B562K160CT" H 6600 5950 60  0001 L CNN "MPN"
+F 4 "Kemet" H 6600 6050 60  0001 L CNN "Manufacturer"
+F 5 "C0402C562K3RACTU" H 6600 5950 60  0001 L CNN "MPN"
 F 6 "5n6" V 6450 5800 50  0000 C CNN "Val"
 	1    6400 5650
@@
 F 2 "sdi-mipi-bridge-footprints:0603-res" H 7250 6400 60  0001 L CNN
 F 3 "" H 7050 6200 50  0001 C CNN
-F 4 "MULTICOMP" H 7250 6600 60  0001 L CNN "Manufacturer"
-F 5 "MCWR06X75R0FTL" H 7250 6500 60  0001 L CNN "MPN"
+F 4 "Yageo" H 7250 6600 60  0001 L CNN "Manufacturer"
+F 5 "RC0603FR-0775RL" H 7250 6500 60  0001 L CNN "MPN"
 F 6 "75R" H 6750 6250 50  0000 L CNN "Val"
 	1    7050 6200
@@
 F 2 "sdi-mipi-bridge-footprints:0603-res" H 6600 6100 60  0001 L CNN
 F 3 "" H 6400 5900 50  0001 C CNN
-F 4 "MULTICOMP" H 6600 6300 60  0001 L CNN "Manufacturer"
-F 5 "MCWR06X75R0FTL" H 6600 6200 60  0001 L CNN "MPN"
+F 4 "Yageo" H 6600 6300 60  0001 L CNN "Manufacturer"
+F 5 "RC0603FR-0775RL" H 6600 6200 60  0001 L CNN "MPN"
 F 6 "75R" H 6550 5850 50  0000 L CNN "Val"
 	1    6400 5900
@@
 F 2 "sdi-mipi-bridge-footprints:0402-res" H 3600 9350 60  0001 L CNN
 F 3 "" H 3400 9150 50  0001 C CNN
-F 4 "VISHAY" H 3600 9550 60  0001 L CNN "Manufacturer"
-F 5 "CRCW0402120KFKED" H 3600 9450 60  0001 L CNN "MPN"
+F 4 "Yageo" H 3600 9550 60  0001 L CNN "Manufacturer"
+F 5 "RC0402FR-07120KL" H 3600 9450 60  0001 L CNN "MPN"
 F 6 "120k" V 3500 9200 50  0000 L CNN "Val"
 	1    3400 9150
@@
 F 2 "sdi-mipi-bridge-footprints:0402-res" H 3600 9900 60  0001 L CNN
 F 3 "" H 3400 9700 50  0001 C CNN
-F 4 "VISHAY" H 3600 10100 60  0001 L CNN "Manufacturer"
-F 5 "CRCW0402120KFKED" H 3600 10000 60  0001 L CNN "MPN"
+F 4 "Yageo" H 3600 10100 60  0001 L CNN "Manufacturer"
+F 5 "RC0402FR-07120KL" H 3600 10000 60  0001 L CNN "MPN"
 F 6 "120k" V 3550 9750 50  0000 L CNN "Val"
 	1    3400 9700
@@
 P 1050 6050
 F 0 "J5" V 950 6000 50  0000 C CNN
-F 1 "MC-HVT1-S04-G" V 1450 6050 50  0000 C CNN
+F 1 "GRPB041VWVN-RC" V 1450 6050 50  0000 C CNN
 F 2 "sdi-mipi-bridge-footprints:PinHeader_1x4_P1.27mm_Drill.7mm" H 1250 6350 60  0001 L CNN
 F 3 "http://www.farnell.com/datasheets/2605295.pdf" H 1250 6450 60  0001 L CNN
-F 4 "MC-HVT1-S04-G" H 1250 6550 60  0001 L CNN "MPN"
-F 5 "Multicomp" H 1250 6650 60  0001 L CNN "Manufacturer"
+F 4 "GRPB041VWVN-RC" H 1250 6550 60  0001 L CNN "MPN"
+F 5 "Sullins" H 1250 6650 60  0001 L CNN "Manufacturer"
 	1    1050 6050
 	0    1    1    0
@@
 F 2 "sdi-mipi-bridge-footprints:SW_SPST_6_Slide_MCDHN-06F-T-V_P1.27mm" H 14250 13700 50  0001 C CNN
 F 3 "" H 14250 13700 50  0001 C CNN
-F 4 "MCDHN-06F-T-V" H 14250 13700 50  0001 C CNN "MPN"
-F 5 "MULTICOMP PRO" H 14250 13700 50  0001 C CNN "Manufacturer"
+F 4 "97C06SRT" H 14250 13700 50  0001 C CNN "MPN"
+F 5 "Grayhill" H 14250 13700 50  0001 C CNN "Manufacturer"
 	1    14250 13700
 	-1   0    0    -1
@@
 F 2 "sdi-mipi-bridge-footprints:SW_SPST_6_Slide_MCDHN-06F-T-V_P1.27mm" H 14250 14650 50  0001 C CNN
 F 3 "" H 14250 14650 50  0001 C CNN
-F 4 "MCDHN-06F-T-V" H 14250 14650 50  0001 C CNN "MPN"
-F 5 "MULTICOMP PRO" H 14250 14650 50  0001 C CNN "Manufacturer"
+F 4 "97C06SRT" H 14250 14650 50  0001 C CNN "MPN"
+F 5 "Grayhill" H 14250 14650 50  0001 C CNN "Manufacturer"
 	1    14250 14650
 	-1   0    0    -1
@@
 P 21100 4150
 F 0 "J4" H 21150 4567 50  0000 C CNN
-F 1 "2199SB-10G-301523" H 21150 4476 50  0000 C CNN
+F 1 "GRPB052VWVN-RC" H 21150 4476 50  0000 C CNN
 F 2 "sdi-mipi-bridge-footprints:PinHeader_2x05_P1.27mm_Vertical" H 21100 4150 50  0001 C CNN
 F 3 "~" H 21100 4150 50  0001 C CNN
-F 4 "2199SB-10G-301523" H 21100 4150 50  0001 C CNN "MPN"
-F 5 "MULTICOMP PRO" H 21100 4150 50  0001 C CNN "Manufacturer"
+F 4 "GRPB052VWVN-RC" H 21100 4150 50  0001 C CNN "MPN"
+F 5 "Sullins" H 21100 4150 50  0001 C CNN "Manufacturer"
 	1    21100 4150
 	1    0    0    -1
@@
 P 1500 5150
 F 0 "J6" H 1550 5567 50  0000 C CNN
-F 1 "2199SB-10G-301523" H 1550 5476 50  0000 C CNN
+F 1 "GRPB052VWVN-RC" H 1550 5476 50  0000 C CNN
 F 2 "sdi-mipi-bridge-footprints:PinHeader_2x05_P1.27mm_Vertical" H 1500 5150 50  0001 C CNN
 F 3 "~" H 1500 5150 50  0001 C CNN
-F 4 "2199SB-10G-301523" H 1500 5150 50  0001 C CNN "MPN"
-F 5 "MULTICOMP PRO" H 1500 5150 50  0001 C CNN "Manufacturer"
+F 4 "GRPB052VWVN-RC" H 1500 5150 50  0001 C CNN "MPN"
+F 5 "Sullins" H 1500 5150 50  0001 C CNN "Manufacturer"
 	1    1500 5150
 	1    0    0    -1

Commit message: Chnage from 12G to 6G BNC connectors
Parts:
- J1, J2: value 031-70526-21 -> 112740-13; MPN 031-70526-21 -> 112740-13
Changed lines of the file:
@@
 P 9150 5350
 F 0 "J2" H 9250 5500 50  0000 L CNN
-F 1 "031-70526-21" H 8500 5200 50  0000 L CNN
+F 1 "112740-13" H 8500 5200 50  0000 L CNN
 F 2 "sdi-mipi-bridge-footprints:BNC_Edge_Conn" H 8910 4520 50  0001 C CNN
-F 3 "https://www.farnell.com/cad/2305565.pdf?_ga=2.190633003.1014497200.1574067480-156563690.1566371002&_gac=1.57062104.1572875319.Cj0KCQiAtf_tBRDtARIsAIbAKe0A1M5y_jdFCiNLNrHM5L2GjmDvn_4qnRvhHAD9jBdL9AmoMNThLCoaAjhJEALw_wcB" H 9010 4620 50  0001 C CNN
-F 4 "031-70526-21" H 9110 4720 51  0001 C CNN "MPN"
+F 3 "" H 9010 4620 50  0001 C CNN
+F 4 "112740-13" H 9110 4720 51  0001 C CNN "MPN"
 F 5 "Amphenol" H 9210 4820 51  0001 C CNN "Manufacturer"
 	1    9150 5350
@@
 P 8550 5650
 F 0 "J1" H 8400 5850 50  0000 L CNN
-F 1 "031-70526-21" H 7900 5500 50  0000 L CNN
+F 1 "112740-13" H 7900 5500 50  0000 L CNN
 F 2 "sdi-mipi-bridge-footprints:BNC_Edge_Conn" H 8310 4820 50  0001 C CNN
-F 3 "https://www.farnell.com/cad/2305565.pdf?_ga=2.190633003.1014497200.1574067480-156563690.1566371002&_gac=1.57062104.1572875319.Cj0KCQiAtf_tBRDtARIsAIbAKe0A1M5y_jdFCiNLNrHM5L2GjmDvn_4qnRvhHAD9jBdL9AmoMNThLCoaAjhJEALw_wcB" H 8410 4920 50  0001 C CNN
-F 4 "031-70526-21" H 8510 5020 51  0001 C CNN "MPN"
+F 3 "" H 8410 4920 50  0001 C CNN
+F 4 "112740-13" H 8510 5020 51  0001 C CNN "MPN"
 F 5 "Amphenol" H 8610 5120 51  0001 C CNN "Manufacturer"
 	1    8550 5650

Commit message: Change C37 from 2n2 to 2u2
Parts:
- C37: value C_2n2_0402 -> C_2u2_0402; symbol sdi-mipi-bridge:C_2n2_0402 -> sdi-mipi-bridge:C_2u2_0402; MPN CGA9N3X7R1C476M230KB -> C0402C225K9PACTU; Manufacturer KEMET -> Kemet; Val 2n2 -> 2u2
Changed lines of the file:
@@
 	8850 9300 8850 9500
 $Comp
-L sdi-mipi-bridge:C_2n2_0402 C37
+L sdi-mipi-bridge:C_2u2_0402 C37
 U 1 1 658AC3D4
 P 8850 9050
 F 0 "C37" H 8965 9095 60  0000 L CNN
-F 1 "C_2n2_0402" H 8850 8900 60  0001 C CNN
+F 1 "C_2u2_0402" H 8850 8900 60  0001 C CNN
 F 2 "sdi-mipi-bridge-footprints:0402-cap" H 9050 9250 60  0001 L CNN
 F 3 "" H 8850 9050 50  0001 C CNN
-F 4 "KEMET" H 9050 9450 60  0001 L CNN "Manufacturer"
-F 5 "CGA9N3X7R1C476M230KB" H 9050 9350 60  0001 L CNN "MPN"
-F 6 "2n2" H 8965 8997 50  0000 L CNN "Val"
+F 4 "Kemet" H 9050 9450 60  0001 L CNN "Manufacturer"
+F 5 "C0402C225K9PACTU" H 9050 9350 60  0001 L CNN "MPN"
+F 6 "2u2" H 8965 8997 50  0000 L CNN "Val"
 	1    8850 9050
 	1    0    0    -1
