File: sdi-mipi-bridge.sch (KiCad schematic (older format))
At the start: 202 parts, among them J1 112740-13, J2 112740-13, J3 WE_68715014522_ONE-SIDE, J4 GRPB052VWVN-RC, J5 GRPB041VWVN-RC, J6 GRPB052VWVN-RC, SW1 SW_DIP_x06, SW2 SW_DIP_x06, U1 MAX8902B, U2 GS2971A, U3 GS2988, U4 CrossLink_LIF-MD6000-6JMG80I, U5 SC18IS602BIPW, Y1 ABM7_27.000MH_D2Y_T

Commit message: Connect PCLK to J7 pin
Connections:
- wire segments 864 -> 862
- no-connect marks 5 -> 7
Changed lines of the file:
@@
 	18000 10350 17000 10350
 Wire Wire Line
-	18000 10150 17000 10150
+	18000 10550 17000 10550
 Text Label 17000 12250 0    50   ~ 0
 DATA_ERRORb
@@
 Text Label 17000 10350 0    50   ~ 0
 H_HSYNC
-Text Label 17000 10150 0    50   ~ 0
+Text Label 17000 10550 0    50   ~ 0
 PCLK
 Wire Wire Line
@@
 Text Label 17300 10750 2    50   ~ 0
 DOUT12
-Text Label 17300 10650 2    50   ~ 0
-DOUT11
-Text Label 17300 10550 2    50   ~ 0
-DOUT10
 Wire Wire Line
 	18000 11450 17000 11450
@@
 Wire Wire Line
 	18000 10750 17000 10750
-Wire Wire Line
-	17000 10650 18000 10650
-Wire Wire Line
-	18000 10550 17000 10550
-Text Label 16900 10650 2    50   ~ 0
+Text Label 16350 10850 0    50   ~ 0
 DOUT[19:10]
 Wire Bus Line
-	16900 10650 16350 10650
-Entry Wire Line
-	17000 10550 16900 10650
-Entry Wire Line
-	17000 10650 16900 10750
+	16900 10850 16350 10850
 Entry Wire Line
 	17000 10750 16900 10850
@@
 	1    0    0    -1
 $EndComp
+NoConn ~ 18000 10150
+NoConn ~ 18000 10650
 Wire Bus Line
-	16900 10650 16900 11550
+	16900 10850 16900 11550
 Wire Bus Line
 	4850 2850 4850 3750

Commit message: Replace DOUT10 and DOUT11 resistors with test pads
Parts:
- removed R7, R8: R_0R_0402, sdi-mipi-bridge-footprints:0402-res, symbol sdi-mipi-bridge:R_0R_0402
- added TP3, TP4: TP_SMD_0_75MM, sdi-mipi-bridge-footprints:Testpoint_smd_0_75mm, symbol sdi-mipi-bridge:TP_SMD_0_75MM
Connections:
- net labels added: DOUT[19:12]
- net labels removed: D10, D11, DOUT10, DOUT11, DOUT[19:10]
- wire segments 862 -> 860
Changed lines of the file:
@@
 Title "SDI-MIPI Bridge"
 Date ""
-Rev "1.1.0"
+Rev "1.2.0"
 Comp ""
 Comment1 "www.antmicro.com"
@@
 Text Label 4350 2950 0    50   ~ 0
 DOUT12
-Text Label 4350 2850 0    50   ~ 0
-DOUT11
-Text Label 4350 2750 0    50   ~ 0
-DOUT10
-Wire Wire Line
-	4250 2750 4750 2750
 Text Label 3550 3650 0    50   ~ 0
 D19
@@
 Text Label 3550 2950 0    50   ~ 0
 D12
-Text Label 3550 2850 0    50   ~ 0
-D11
-Text Label 3550 2750 0    50   ~ 0
-D10
 Text Label 3550 2650 0    50   ~ 0
 D9
@@
 	3900 2650 3550 2650
 Wire Wire Line
-	3950 2750 3550 2750
-Wire Wire Line
 	3550 3050 3950 3050
 Wire Wire Line
-	3550 2850 3950 2850
-Wire Wire Line
 	3950 2950 3550 2950
 Wire Wire Line
@@
 	4750 2950 4250 2950
 Wire Wire Line
-	4750 2850 4250 2850
-Wire Wire Line
 	3550 2450 3900 2450
 Wire Wire Line
@@
 Entry Wire Line
 	4750 2950 4850 3050
-Entry Wire Line
-	4750 2850 4850 2950
-Entry Wire Line
-	4750 2750 4850 2850
 Wire Bus Line
-	4850 2850 5400 2850
+	4850 3050 5400 3050
 $Comp
 L sdi-mipi-bridge:TP_SMD1MM TP2
@@
 Wire Wire Line
 	8150 2800 8800 2800
-Text Label 4900 2850 0    50   ~ 0
-DOUT[19:10]
+Text Label 4900 3050 0    50   ~ 0
+DOUT[19:12]
 Wire Wire Line
 	10850 1800 10850 1700
@@
 $EndComp
 $Comp
-L sdi-mipi-bridge:R_0R_0402 R7
-U 1 1 5DED67D1
-P 4100 2750
-F 0 "R7" H 4300 2800 60  0000 C CNN
-F 1 "R_0R_0402" H 4100 2600 60  0001 C CNN
-F 2 "sdi-mipi-bridge-footprints:0402-res" H 4300 2950 60  0001 L CNN
-F 3 "" H 4100 2750 50  0001 C CNN
-F 4 "PANASONIC" H 4300 3150 60  0001 L CNN "Manufacturer"
-F 5 "ERJ2GE0R00X" H 4300 3050 60  0001 L CNN "MPN"
-F 6 "0R" H 4100 2750 50  0000 C CNN "Val"
-	1    4100 2750
-	-1   0    0    -1
-$EndComp
-$Comp
-L sdi-mipi-bridge:R_0R_0402 R8
-U 1 1 5DED76DC
-P 4100 2850
-F 0 "R8" H 4300 2900 60  0000 C CNN
-F 1 "R_0R_0402" H 4100 2700 60  0001 C CNN
-F 2 "sdi-mipi-bridge-footprints:0402-res" H 4300 3050 60  0001 L CNN
-F 3 "" H 4100 2850 50  0001 C CNN
-F 4 "PANASONIC" H 4300 3250 60  0001 L CNN "Manufacturer"
-F 5 "ERJ2GE0R00X" H 4300 3150 60  0001 L CNN "MPN"
-F 6 "0R" H 4100 2850 50  0000 C CNN "Val"
-	1    4100 2850
-	-1   0    0    -1
-$EndComp
-$Comp
 L sdi-mipi-bridge:R_0R_0402 R9
 U 1 1 5DED86FD
@@
 	18000 10750 17000 10750
 Text Label 16350 10850 0    50   ~ 0
-DOUT[19:10]
+DOUT[19:12]
 Wire Bus Line
 	16900 10850 16350 10850
@@
 NoConn ~ 18000 10150
 NoConn ~ 18000 10650
+Wire Wire Line
+	3900 2750 3550 2750
+Wire Wire Line
+	3900 2850 3550 2850
+$Comp
+L sdi-mipi-bridge:TP_SMD_0_75MM TP3
+U 1 1 60D6CAD4
+P 4000 2750
+F 0 "TP3" V 4000 2700 50  0000 R CNN
+F 1 "TP_SMD_0_75MM" H 4000 2650 50  0001 C CNN
+F 2 "sdi-mipi-bridge-footprints:Testpoint_smd_0_75mm" H 4200 2950 60  0001 L CNN
+F 3 "" H 4200 3050 60  0001 L CNN
+	1    4000 2750
+	0    -1   -1   0
+$EndComp
+$Comp
+L sdi-mipi-bridge:TP_SMD_0_75MM TP4
+U 1 1 60D6CADA
+P 4000 2850
+F 0 "TP4" V 4000 2800 50  0000 R CNN
+F 1 "TP_SMD_0_75MM" H 4000 2750 50  0001 C CNN
+F 2 "sdi-mipi-bridge-footprints:Testpoint_smd_0_75mm" H 4200 3050 60  0001 L CNN
+F 3 "" H 4200 3150 60  0001 L CNN
+	1    4000 2850
+	0    -1   -1   0
+$EndComp
 Wire Bus Line
-	16900 10850 16900 11550
+	4850 3050 4850 3750
 Wire Bus Line
-	4850 2850 4850 3750
+	16900 10850 16900 11550
 $EndSCHEMATC

Commit message: Add DNP field to SDA_CL resistors
Parts:
- R37, R38: DNP (none) -> 1
Changed lines of the file:
@@
 F 5 "ERJ2GE0R00X" H 17350 5250 60  0001 L CNN "MPN"
 F 6 "0R" H 17150 4950 50  0000 C CNN "Val"
+F 7 "1" H 17150 4950 50  0001 C CNN "DNP"
 	1    17150 4950
 	-1   0    0    -1
@@
 F 5 "ERJ2GE0R00X" H 17350 5350 60  0001 L CNN "MPN"
 F 6 "0R" H 17150 5050 50  0000 C CNN "Val"
+F 7 "1" H 17150 5050 50  0001 C CNN "DNP"
 	1    17150 5050
 	-1   0    0    -1
@@
 	1    0    0    -1
 $EndComp
-NoConn ~ 18000 10150
 NoConn ~ 18000 10650
 Wire Wire Line
@@
 Wire Bus Line
 	16900 10850 16900 11550
+NoConn ~ 18000 10150
 $EndSCHEMATC
