File: sdi-mipi-bridge.sch (KiCad schematic (older format))
At the start: 202 parts, among them J1 112740-13, J2 112740-13, J3 WE_68715014522_ONE-SIDE, J4 GRPB052VWVN-RC, J5 GRPB041VWVN-RC, J6 GRPB052VWVN-RC, SW1 SW_DIP_x06, SW2 SW_DIP_x06, U1 MAX8902B, U2 GS2971A, U3 GS2988, U4 CrossLink_LIF-MD6000-6JMG80I, U5 SC18IS602BIPW, Y1 ABM7_27.000MH_D2Y_T

Commit message: Add 0R resistor on 3.3v input to allow FFC to be disconnected from net
Parts:
- added R92: R_0R_0402, sdi-mipi-bridge-footprints:0402-res, symbol sdi-mipi-bridge:R_0R_0402
Connections:
- wire segments 864 -> 866
Changed lines of the file:
@@
 MIPI0_CLK_N
 Wire Wire Line
-	18150 6050 17750 6050
-Wire Wire Line
-	18150 5950 17750 5950
+	18150 5950 18050 5950
 Connection ~ 17500 3950
-Connection ~ 17750 5950
-Wire Wire Line
-	17750 6050 17750 5950
 Connection ~ 17500 4250
 Wire Wire Line
@@
 Wire Wire Line
 	18150 2150 17500 2150
-Wire Wire Line
-	17750 5850 17750 5950
 $Comp
 L sdi-mipi-bridge:GNDREF #PWR?
@@
 L sdi-mipi-bridge:+3V3 #PWR0130
 U 1 1 5F104E29
-P 17750 5850
-F 0 "#PWR0130" H 17750 5700 50  0001 C CNN
-F 1 "+3.3V" H 17765 6023 50  0000 C CNN
-F 2 "" H 17750 5850 50  0001 C CNN
-F 3 "" H 17750 5850 50  0001 C CNN
-	1    17750 5850
+P 16750 5850
+F 0 "#PWR0130" H 16750 5700 50  0001 C CNN
+F 1 "+3.3V" H 16765 6023 50  0000 C CNN
+F 2 "" H 16750 5850 50  0001 C CNN
+F 3 "" H 16750 5850 50  0001 C CNN
+	1    16750 5850
 	1    0    0    -1
 $EndComp
@@
 Entry Wire Line
 	17000 10150 16900 10250
+$Comp
+L sdi-mipi-bridge:R_0R_0402 R92
+U 1 1 5FF458A2
+P 17150 5950
+F 0 "R92" H 17400 6000 60  0000 C CNN
+F 1 "R_0R_0402" H 17150 5800 60  0001 C CNN
+F 2 "sdi-mipi-bridge-footprints:0402-res" H 17350 6150 60  0001 L CNN
+F 3 "" H 17150 5950 50  0001 C CNN
+F 4 "PANASONIC" H 17350 6350 60  0001 L CNN "Manufacturer"
+F 5 "ERJ2GE0R00X" H 17350 6250 60  0001 L CNN "MPN"
+F 6 "0R" H 17150 5950 50  0000 C CNN "Val"
+	1    17150 5950
+	-1   0    0    -1
+$EndComp
+Wire Wire Line
+	16750 5850 16750 5950
+Wire Wire Line
+	16750 5950 17000 5950
+Wire Wire Line
+	18150 6050 18050 6050
+Wire Wire Line
+	18050 6050 18050 5950
+Connection ~ 18050 5950
+Wire Wire Line
+	17300 5950 18050 5950
+Text Notes 17250 4950 0    50   ~ 10
+DNP
+Text Notes 17250 5050 0    50   ~ 10
+DNP
 Wire Bus Line
 	16900 10250 16900 11550

Commit message: Change RST pullup from 2k2 to 4k7 and note I2C pull-ups as DNP
Parts:
- R84: value R_2k2_0402 -> R_4k7_0402; symbol sdi-mipi-bridge:R_2k2_0402 -> sdi-mipi-bridge:R_4k7_0402; MPN RC0402FR-072K2L -> ERJ2GEJ472X; Manufacturer YAGEO -> PANASONIC_ELECTRONIC_COMPONENTS; Val 2k2 -> 4k7
Changed lines of the file:
@@
 	14750 5950 14750 6100
 $Comp
-L sdi-mipi-bridge:R_2k2_0402 R84
+L sdi-mipi-bridge:R_4k7_0402 R84
 U 1 1 5F55ED44
 P 14750 6250
 F 0 "R84" V 14600 6050 60  0000 L CNN
-F 1 "R_2k2_0402" H 14750 6100 60  0001 C CNN
+F 1 "R_4k7_0402" H 14750 6100 60  0001 C CNN
 F 2 "sdi-mipi-bridge-footprints:0402-res" H 14950 6450 60  0001 L CNN
 F 3 "" H 14750 6250 50  0001 C CNN
-F 4 "YAGEO" H 14950 6650 60  0001 L CNN "Manufacturer"
-F 5 "RC0402FR-072K2L" H 14950 6550 60  0001 L CNN "MPN"
-F 6 "2k2" V 14900 6300 50  0000 L CNN "Val"
+F 4 "PANASONIC_ELECTRONIC_COMPONENTS" H 14950 6650 60  0001 L CNN "Manufacturer"
+F 5 "ERJ2GEJ472X" H 14950 6550 60  0001 L CNN "MPN"
+F 6 "4k7" V 14900 6300 50  0000 L CNN "Val"
 	1    14750 6250
 	0    1    1    0
@@
 Wire Bus Line
 	4850 2850 4850 3750
+Text Notes 21450 6300 0    50   ~ 10
+DNP
+Text Notes 21200 6300 0    50   ~ 10
+DNP
+Text Notes 20950 6300 0    50   ~ 10
+DNP
+Text Notes 20700 6300 0    50   ~ 10
+DNP
 $EndSCHEMATC

Commit message: Connect CRESET_B to GPIO2 from U5
Connections:
- wire segments 866 -> 867
- no-connect marks 5 -> 4
Changed lines of the file:
@@
 Wire Wire Line
 	19350 1200 19350 1450
-NoConn ~ 21850 1800
 NoConn ~ 21850 2100
 NoConn ~ 20250 1800
@@
 Text Notes 20700 6300 0    50   ~ 10
 DNP
+Text Label 22550 1800 2    50   ~ 0
+CRESET_B
+Wire Wire Line
+	21850 1800 22550 1800
 Wire Bus Line
 	16900 10250 16900 11550

Commit message: Connect configuration I2C from U4 to J3
Parts:
- added R97, R98: R_0R_0402, sdi-mipi-bridge-footprints:0402-res, symbol sdi-mipi-bridge:R_0R_0402
Connections:
- wire segments 867 -> 871

Commit message: Reuse R37,R38 to reconnect configuration I2C
Parts:
- removed R97, R98: R_0R_0402, sdi-mipi-bridge-footprints:0402-res, symbol sdi-mipi-bridge:R_0R_0402
Connections:
- wire segments 871 -> 867
Changed lines of the file:
@@
 Text Label 18150 5150 2    50   ~ 0
 SDA1
-Text Label 16450 5250 0    50   ~ 0
+Text Label 16225 5250 0    50   ~ 0
 SCL_GS
-Text Label 16450 5150 0    50   ~ 0
+Text Label 16225 5150 0    50   ~ 0
 SDA_GS
-Text Label 16450 5050 0    50   ~ 0
-SCL_CL
-Text Label 16450 4950 0    50   ~ 0
-SDA_CL
 Text Label 18150 5350 2    50   ~ 0
 SDA2
 Text Label 18150 5450 2    50   ~ 0
 SCL2
-Text Label 16450 5450 0    50   ~ 0
-SCL_CL
-Text Label 16450 5350 0    50   ~ 0
-SDA_CL
 Wire Wire Line
 	17750 5050 17750 5250
@@
 	-1   0    0    -1
 $EndComp
-$Comp
-L sdi-mipi-bridge:R_0R_0402 R42
-U 1 1 61725908
-P 17150 5450
-F 0 "R42" H 17400 5500 60  0000 C CNN
-F 1 "R_0R_0402" H 17150 5300 60  0001 C CNN
-F 2 "sdi-mipi-bridge-footprints:0402-res" H 17350 5650 60  0001 L CNN
-F 3 "" H 17150 5450 50  0001 C CNN
-F 4 "PANASONIC" H 17350 5850 60  0001 L CNN "Manufacturer"
-F 5 "ERJ2GE0R00X" H 17350 5750 60  0001 L CNN "MPN"
-F 6 "0R" H 17150 5450 50  0000 C CNN "Val"
-	1    17150 5450
-	-1   0    0    -1
-$EndComp
-$Comp
-L sdi-mipi-bridge:R_0R_0402 R41
-U 1 1 617258FF
-P 17150 5350
-F 0 "R41" H 17400 5400 60  0000 C CNN
-F 1 "R_0R_0402" H 17150 5200 60  0001 C CNN
-F 2 "sdi-mipi-bridge-footprints:0402-res" H 17350 5550 60  0001 L CNN
-F 3 "" H 17150 5350 50  0001 C CNN
-F 4 "PANASONIC" H 17350 5750 60  0001 L CNN "Manufacturer"
-F 5 "ERJ2GE0R00X" H 17350 5650 60  0001 L CNN "MPN"
-F 6 "0R" H 17150 5350 50  0000 C CNN "Val"
-	1    17150 5350
-	-1   0    0    -1
-$EndComp
-Wire Wire Line
-	16450 5450 17000 5450
-Wire Wire Line
-	16450 5350 17000 5350
-Wire Wire Line
-	16450 5250 17000 5250
-Wire Wire Line
-	16450 5150 17000 5150
-Wire Wire Line
-	16450 5050 17000 5050
-Wire Wire Line
-	16450 4950 17000 4950
+Wire Wire Line
+	16225 5250 17000 5250
+Wire Wire Line
+	16225 5150 17000 5150
+Wire Wire Line
+	16225 5050 17000 5050
+Wire Wire Line
+	16225 4950 17000 4950
 Wire Wire Line
 	17300 5250 17750 5250
@@
 Wire Wire Line
 	17300 4950 17850 4950
-Text Notes 16150 4750 0    39   ~ 0
-CrossLink and Semtech at same I2C Line
-Wire Notes Line style dash_dot
-	16100 4650 16100 5050
-Wire Notes Line style dash_dot
-	17450 5050 16100 5050
-Wire Notes Line style dash_dot
-	17450 5050 17450 4650
-Wire Notes Line style dash_dot
-	17450 4650 16100 4650
 Wire Notes Line style dash_dot
 	19650 5900 19650 6450
@@
 Wire Wire Line
 	17300 5950 18050 5950
-Text Notes 17250 4950 0    50   ~ 10
+Text Notes 17275 5350 0    50   ~ 10
 DNP
-Text Notes 17250 5050 0    50   ~ 10
+Text Notes 17275 5450 0    50   ~ 10
 DNP
 Text Notes 21450 6300 0    50   ~ 10
@@
 Wire Wire Line
 	21850 1800 22550 1800
-Text Label 625  5325 0    50   ~ 0
+Wire Wire Line
+	16225 5450 17000 5450
+Wire Wire Line
+	16225 5350 17000 5350
+$Comp
+L sdi-mipi-bridge:R_0R_0402 R42
+U 1 1 61725908
+P 17150 5450
+F 0 "R42" H 17400 5500 60  0000 C CNN
+F 1 "R_0R_0402" H 17150 5300 60  0001 C CNN
+F 2 "sdi-mipi-bridge-footprints:0402-res" H 17350 5650 60  0001 L CNN
+F 3 "" H 17150 5450 50  0001 C CNN
+F 4 "PANASONIC" H 17350 5850 60  0001 L CNN "Manufacturer"
+F 5 "ERJ2GE0R00X" H 17350 5750 60  0001 L CNN "MPN"
+F 6 "0R" H 17150 5450 50  0000 C CNN "Val"
+	1    17150 5450
+	-1   0    0    -1
+$EndComp
+$Comp
+L sdi-mipi-bridge:R_0R_0402 R41
+U 1 1 617258FF
+P 17150 5350
+F 0 "R41" H 17400 5400 60  0000 C CNN
+F 1 "R_0R_0402" H 17150 5200 60  0001 C CNN
+F 2 "sdi-mipi-bridge-footprints:0402-res" H 17350 5550 60  0001 L CNN
+F 3 "" H 17150 5350 50  0001 C CNN
+F 4 "PANASONIC" H 17350 5750 60  0001 L CNN "Manufacturer"
+F 5 "ERJ2GE0R00X" H 17350 5650 60  0001 L CNN "MPN"
+F 6 "0R" H 17150 5350 50  0000 C CNN "Val"
+	1    17150 5350
+	-1   0    0    -1
+$EndComp
+Wire Notes Line style dash_dot
+	16100 4650 16100 5050
+Wire Notes Line style dash_dot
+	17450 5050 16100 5050
+Wire Notes Line style dash_dot
+	17450 5050 17450 4650
+Wire Notes Line style dash_dot
+	17450 4650 16100 4650
+Text Notes 16150 4750 0    39   ~ 0
+CrossLink and Semtech at same I2C Line
+Text Label 16225 5350 0    50   ~ 0
 SPI_SCK(SDA)
-Text Label 625  5475 0    50   ~ 0
+Text Label 16225 4950 0    50   ~ 0
+SPI_SCK(SDA)
+Text Label 16225 5050 0    50   ~ 0
 SPI_SS(SCL)
-$Comp
-L sdi-mipi-bridge:R_0R_0402 R?
-U 1 1 609716DE
-P 1425 5325
-AR Path="/5DD55102/609716DE" Ref="R?"  Part="1"
-AR Path="/609716DE" Ref="R97"  Part="1"
-F 0 "R97" H 1600 5275 60  0000 C CNN
-F 1 "R_0R_0402" H 1425 5175 60  0001 C CNN
-F 2 "sdi-mipi-bridge-footprints:0402-res" H 1625 5525 60  0001 L CNN
-F 3 "" H 1425 5325 50  0001 C CNN
-F 4 "PANASONIC" H 1625 5725 60  0001 L CNN "Manufacturer"
-F 5 "ERJ2GE0R00X" H 1625 5625 60  0001 L CNN "MPN"
-F 6 "0R" H 1425 5325 50  0000 C CNN "Val"
-	1    1425 5325
-	-1   0    0    1
-$EndComp
-$Comp
-L sdi-mipi-bridge:R_0R_0402 R?
-U 1 1 60972551
-P 1425 5475
-AR Path="/5DD55102/60972551" Ref="R?"  Part="1"
-AR Path="/60972551" Ref="R98"  Part="1"
-F 0 "R98" H 1600 5425 60  0000 C CNN
-F 1 "R_0R_0402" H 1425 5325 60  0001 C CNN
-F 2 "sdi-mipi-bridge-footprints:0402-res" H 1625 5675 60  0001 L CNN
-F 3 "" H 1425 5475 50  0001 C CNN
-F 4 "PANASONIC" H 1625 5875 60  0001 L CNN "Manufacturer"
-F 5 "ERJ2GE0R00X" H 1625 5775 60  0001 L CNN "MPN"
-F 6 "0R" H 1425 5475 50  0000 C CNN "Val"
-	1    1425 5475
-	-1   0    0    1
-$EndComp
-Wire Wire Line
-	1275 5325 625  5325
-Wire Wire Line
-	1275 5475 625  5475
-Wire Wire Line
-	1575 5325 2100 5325
-Wire Wire Line
-	1575 5475 2100 5475
+Text Label 16225 5450 0    50   ~ 0
+SPI_SS(SCL)
 Wire Bus Line
 	16900 10250 16900 11550
 Wire Bus Line
 	4850 2850 4850 3750
-Text Label 2100 5325 2    50   ~ 0
-SDA_GS
-Text Label 2100 5475 2    50   ~ 0
-SCL_GS
 $EndSCHEMATC

Commit message: Update layout DRC-clean
Connections:
- net labels removed: SCL_CL, SDA_CL
Changed lines of the file:
@@
 Wire Wire Line
 	20650 6350 20650 6800
-Text Label 21900 6800 0    50   ~ 0
-SCL_CL
-Text Label 21900 6700 0    50   ~ 0
-SDA_CL
 Wire Wire Line
 	21400 5700 21400 5750
@@
 Wire Bus Line
 	4850 2850 4850 3750
+Text Label 21900 6700 0    50   ~ 0
+SPI_SCK(SDA)
+Text Label 21900 6800 0    50   ~ 0
+SPI_SS(SCL)
 $EndSCHEMATC

Commit message: Update DNP attributes
Parts:
- R32, R34: DNP 1 -> DNP
- R37, R38: DNP 1 -> (none)
- R41, R42, R85, R86, R87, R94: DNP (none) -> DNP
Changed lines of the file:
@@
 U 1 1 5DFFCF9B
 P 14650 3150
-F 0 "R32" H 14550 3250 60  0000 C CNN
+F 0 "R32" H 14625 3325 60  0000 C CNN
 F 1 "R_0R_0402" H 14650 3000 60  0001 C CNN
 F 2 "sdi-mipi-bridge-footprints:0402-res" H 14850 3350 60  0001 L CNN
@@
 F 4 "PANASONIC" H 14850 3550 60  0001 L CNN "Manufacturer"
 F 5 "ERJ2GE0R00X" H 14850 3450 60  0001 L CNN "MPN"
-F 6 "0R" H 14650 3150 50  0000 C CNN "Val"
-F 7 "1" H 14650 3150 50  0001 C CNN "DNP"
+F 6 "0R" H 14650 3150 50  0001 C CNN "Val"
+F 7 "DNP" H 14625 3250 50  0000 C CNN "DNP"
 	1    14650 3150
 	1    0    0    -1
@@
 U 1 1 5DFFCE31
 P 15200 2850
-F 0 "R34" V 15050 2650 60  0000 L CNN
+F 0 "R34" V 15175 2625 60  0000 L CNN
 F 1 "R_0R_0402" H 15200 2700 60  0001 C CNN
 F 2 "sdi-mipi-bridge-footprints:0402-res" H 15400 3050 60  0001 L CNN
@@
 F 4 "PANASONIC" H 15400 3250 60  0001 L CNN "Manufacturer"
 F 5 "ERJ2GE0R00X" H 15400 3150 60  0001 L CNN "MPN"
-F 6 "0R" V 15350 2900 50  0000 L CNN "Val"
-F 7 "1" V 15200 2850 50  0001 C CNN "DNP"
+F 6 "0R" V 15350 2900 50  0001 L CNN "Val"
+F 7 "DNP" V 15250 2700 50  0000 C CNN "DNP"
 	1    15200 2850
 	0    1    1    0
@@
 F 5 "ERJ2GE0R00X" H 17350 5250 60  0001 L CNN "MPN"
 F 6 "0R" H 17150 4950 50  0000 C CNN "Val"
-F 7 "1" H 17150 4950 50  0001 C CNN "DNP"
 	1    17150 4950
 	-1   0    0    -1
@@
 F 5 "ERJ2GE0R00X" H 17350 5350 60  0001 L CNN "MPN"
 F 6 "0R" H 17150 5050 50  0000 C CNN "Val"
-F 7 "1" H 17150 5050 50  0001 C CNN "DNP"
 	1    17150 5050
 	-1   0    0    -1
@@
 	1    0    0    -1
 $EndComp
-Text Notes 15300 2850 0    50   ~ 10
-DNP
-Text Notes 14750 3050 0    50   ~ 10
-DNP
 Wire Wire Line
 	2050 9200 1950 9200
@@
 F 4 "YAGEO" H 20850 6600 60  0001 L CNN "Manufacturer"
 F 5 "RC0402FR-072K2L" H 20850 6500 60  0001 L CNN "MPN"
-F 6 "2k2" V 20800 6250 50  0000 L CNN "Val"
+F 6 "2k2" V 20800 6250 50  0001 L CNN "Val"
+F 7 "DNP" V 20700 6325 50  0000 C CNN "DNP"
 	1    20650 6200
 	0    1    1    0
@@
 F 4 "YAGEO" H 21100 6600 60  0001 L CNN "Manufacturer"
 F 5 "RC0402FR-072K2L" H 21100 6500 60  0001 L CNN "MPN"
-F 6 "2k2" V 21050 6250 50  0000 L CNN "Val"
+F 6 "2k2" V 21050 6250 50  0001 L CNN "Val"
+F 7 "DNP" V 20950 6325 50  0000 C CNN "DNP"
 	1    20900 6200
 	0    1    1    0
@@
 F 4 "YAGEO" H 21350 6600 60  0001 L CNN "Manufacturer"
 F 5 "RC0402FR-072K2L" H 21350 6500 60  0001 L CNN "MPN"
-F 6 "2k2" V 21300 6250 50  0000 L CNN "Val"
+F 6 "2k2" V 21300 6250 50  0001 L CNN "Val"
+F 7 "DNP" V 21200 6325 50  0000 C CNN "DNP"
 	1    21150 6200
 	0    1    1    0
 $EndComp
-$Comp
-L sdi-mipi-bridge:R_2k2_0402 R94
-U 1 1 5FB2B4FD
-P 21400 6200
-F 0 "R94" V 21250 6000 60  0000 L CNN
-F 1 "R_2k2_0402" H 21400 6050 60  0001 C CNN
-F 2 "sdi-mipi-bridge-footprints:0402-res" H 21600 6400 60  0001 L CNN
-F 3 "" H 21400 6200 50  0001 C CNN
-F 4 "YAGEO" H 21600 6600 60  0001 L CNN "Manufacturer"
-F 5 "RC0402FR-072K2L" H 21600 6500 60  0001 L CNN "MPN"
-F 6 "2k2" V 21550 6250 50  0000 L CNN "Val"
-	1    21400 6200
-	0    1    1    0
-$EndComp
 Wire Wire Line
 	14750 5950 14750 6100
@@
 Wire Wire Line
 	17300 5950 18050 5950
-Text Notes 17275 5350 0    50   ~ 10
-DNP
-Text Notes 17275 5450 0    50   ~ 10
-DNP
-Text Notes 21450 6300 0    50   ~ 10
-DNP
-Text Notes 21200 6300 0    50   ~ 10
-DNP
-Text Notes 20950 6300 0    50   ~ 10
-DNP
-Text Notes 20700 6300 0    50   ~ 10
-DNP
 Text Label 22550 1800 2    50   ~ 0
 CRESET_B
@@
 F 4 "PANASONIC" H 17350 5850 60  0001 L CNN "Manufacturer"
 F 5 "ERJ2GE0R00X" H 17350 5750 60  0001 L CNN "MPN"
-F 6 "0R" H 17150 5450 50  0000 C CNN "Val"
+F 6 "0R" H 17150 5450 50  0001 C CNN "Val"
+F 7 "DNP" H 16925 5500 50  0000 C CNN "DNP"
 	1    17150 5450
 	-1   0    0    -1
@@
 F 4 "PANASONIC" H 17350 5750 60  0001 L CNN "Manufacturer"
 F 5 "ERJ2GE0R00X" H 17350 5650 60  0001 L CNN "MPN"
-F 6 "0R" H 17150 5350 50  0000 C CNN "Val"
+F 6 "0R" H 17150 5350 50  0001 C CNN "Val"
+F 7 "DNP" H 16925 5400 50  0000 C CNN "DNP"
 	1    17150 5350
 	-1   0    0    -1
@@
 Text Label 16225 5450 0    50   ~ 0
 SPI_SS(SCL)
-Wire Bus Line
-	16900 10250 16900 11550
-Wire Bus Line
-	4850 2850 4850 3750
 Text Label 21900 6700 0    50   ~ 0
 SPI_SCK(SDA)
 Text Label 21900 6800 0    50   ~ 0
 SPI_SS(SCL)
+Wire Bus Line
+	16900 10250 16900 11550
+Wire Bus Line
+	4850 2850 4850 3750
+$Comp
+L sdi-mipi-bridge:R_2k2_0402 R94
+U 1 1 5FB2B4FD
+P 21400 6200
+F 0 "R94" V 21250 6000 60  0000 L CNN
+F 1 "R_2k2_0402" H 21400 6050 60  0001 C CNN
+F 2 "sdi-mipi-bridge-footprints:0402-res" H 21600 6400 60  0001 L CNN
+F 3 "" H 21400 6200 50  0001 C CNN
+F 4 "YAGEO" H 21600 6600 60  0001 L CNN "Manufacturer"
+F 5 "RC0402FR-072K2L" H 21600 6500 60  0001 L CNN "MPN"
+F 6 "2k2" V 21550 6250 50  0001 L CNN "Val"
+F 7 "DNP" V 21450 6325 50  0000 C CNN "DNP"
+	1    21400 6200
+	0    1    1    0
+$EndComp
 $EndSCHEMATC
