File: sdi-mipi-bridge.kicad_sch (KiCad schematic)
At the start: 186 parts, among them J1 112740-13, J2 112740-13, J3 WE_68715014522_ONE-SIDE, J4 GRPB052VWVN-RC, J5 GRPB041VWVN-RC, J6 GRPB052VWVN-RC, U1 MAX8902B, U2 GS2971A, U3 GS2988, U4 CrossLink_LIF-MD6000-6JMG80I, U5 SC18IS602BIPW, Y1 ABM7_27.000MH_D2Y_T

Commit message: Applied globlib
Parts:
- C1, C15: footprint sdi-mipi-bridge-footprints:0603-cap -> antmicro-footprints:C_0603_1608Metric; symbol sdi-mipi-bridge:C_10u_0603 -> antmicroCapacitors0603:C_10u_0603
- C10, C11, C12, C13, C14, C16, C17, C18, C19, C2, C20, C21, C22, C3, C32, C33, C34, C36, C4, C5, C6, C65, C7, C8, C9: footprint sdi-mipi-bridge-footprints:0402-cap -> antmicro-footprints:C_0402_1005Metric; symbol sdi-mipi-bridge:C_10n_0402 -> antmicroCapacitors0402:C_10n_0402
- C23, C31, C42, C52: footprint sdi-mipi-bridge-footprints:0402-cap -> antmicro-footprints:C_0402_1005Metric; symbol sdi-mipi-bridge:C_4u7_0402 -> antmicroCapacitors0402:C_4u7_0402
- C24, C25, C26, C28, C29, C30, C35, C45, C47, C55, C56, C62: footprint sdi-mipi-bridge-footprints:0402-cap -> antmicro-footprints:C_0402_1005Metric; symbol sdi-mipi-bridge:C_1u_0402 -> antmicroCapacitors0402:C_1u_0402
- C27: footprint sdi-mipi-bridge-footprints:0402-res -> antmicro-footprints:C_0402_1005Metric; symbol sdi-mipi-bridge:C_5n6_0402 -> antmicroCapacitors0402:C_5n6_0402
- C37, C38: footprint sdi-mipi-bridge-footprints:0402-cap -> antmicro-footprints:C_0402_1005Metric; symbol sdi-mipi-bridge:C_2u2_0402 -> antmicroCapacitors0402:C_2u2_0402
- C39, C40, C41, C44, C46, C48, C49, C50, C51, C53, C54, C57: footprint sdi-mipi-bridge-footprints:0402-cap -> antmicro-footprints:C_0402_1005Metric; symbol sdi-mipi-bridge:C_100n_0402_6V3 -> antmicroCapacitorsmisc:C_100n_6V3_0402
- C43: footprint sdi-mipi-bridge-footprints:0603-res -> antmicro-footprints:C_0603_1608Metric; symbol sdi-mipi-bridge:C_6n2_0603 -> antmicroCapacitors0603:C_6n2_0603
- C58: footprint sdi-mipi-bridge-footprints:0603-cap -> antmicro-footprints:C_0603_1608Metric; symbol sdi-mipi-bridge:C_33u_0603 -> antmicroCapacitorspol:C_33u_0603
- C59, C60: footprint sdi-mipi-bridge-footprints:0402-res -> antmicro-footprints:C_0402_1005Metric; symbol sdi-mipi-bridge:C_16p_0402 -> antmicroCapacitors0402:C_16p_0402
- C61, C64: footprint sdi-mipi-bridge-footprints:0402-cap -> antmicro-footprints:C_0402_1005Metric; symbol sdi-mipi-bridge:C_470n_0402 -> antmicroCapacitors0402:C_470n_0402
- C63: footprint sdi-mipi-bridge-footprints:0402-cap -> antmicro-footprints:C_0402_1005Metric; symbol sdi-mipi-bridge:C_47n_0402 -> antmicroCapacitors0402:C_47n_0402
- D1, D2, D4, D5: footprint sdi-mipi-bridge-footprints:LED_0603 -> antmicro-footprints:LED_0603_1608Metric_G; symbol sdi-mipi-bridge:LG_L29K-G2J1-24-Z -> antmicroLEDIndicationDiscrete:LED_G_0603_LG_L29K-G2J1-24-Z
- FB1, FB2, FB3: footprint sdi-mipi-bridge-footprints:0603-res -> antmicro-footprints:FB_0603_1608Metric; symbol sdi-mipi-bridge:BLM18PG121SN1D -> antmicroFerriteBeadsandChips:FB_120Z_2A_0603
- J1, J2: footprint sdi-mipi-bridge-footprints:BNC_Edge_Conn -> antmicro-footprints:Conn_BNC_031-70526-21; symbol sdi-mipi-bridge:031-70526-21 -> antmicroCoaxialConnectorsRF:Conn_BNC_031-70526-21
- J3: footprint sdi-mipi-bridge-footprints:WE_68715014522_ONE-SIDE -> antmicro-footprints:WE_68715014522_ONE-SIDE; symbol sdi-mipi-bridge:WE_68715014522_ONE-SIDE -> antmicroFCCConnectors:Conn_FFC_68715014522_ONE-SIDE
- J4, J6: footprint sdi-mipi-bridge-footprints:PinHeader_2x05_P1.27mm_Vertical -> antmicro-footprints:PinHeader_2x05_P1.27mm_Vertical; symbol sdi-mipi-bridge:2199SB-10G-301523 -> antmicroRectangularConnectorsHeadersMalePins:2199SB-10G-301523
- J5: footprint sdi-mipi-bridge-footprints:PinHeader_1x4_P1.27mm_Drill.7mm -> antmicro-footprints:PinHeader_1x4_P1.27mm_Drill.7mm; symbol sdi-mipi-bridge:MC-HVT1-S04-G -> antmicroRectangularConnectorsHeadersMalePins:MC-HVT1-S04-G
- N1: footprint sdi-mipi-bridge-footprints:antmicro-logo_scaled_20mm -> antmicro-footprints:antmicro-logo; symbol sdi-mipi-bridge:antmicro_logo -> antmicroMechanicalParts:antmicro_logo
- N2: footprint sdi-mipi-bridge-footprints:oshw-logo -> antmicro-footprints:oshw-logo; symbol sdi-mipi-bridge:oshw_logo -> antmicroMechanicalParts:oshw_logo
- R1, R2, R3: footprint sdi-mipi-bridge-footprints:0402-res -> antmicro-footprints:R_0402_1005Metric; symbol sdi-mipi-bridge:R_22R_0402 -> antmicroResistors0402:R_22R_0402
- R100, R101, R102, R103, R104, R106, R107, R108, R109, R110, R111, R65, R66, R68, R75, R76, R77, R78, R79, R80, R81, R83, R84, R97, R98, R99: footprint sdi-mipi-bridge-footprints:0402-res -> antmicro-footprints:R_0402_1005Metric; symbol sdi-mipi-bridge:R_10k_0402 -> antmicroResistors0402:R_10k_0402
- R105, R21, R22, R23, R24, R25, R26, R31, R32, R34, R37, R38, R39, R40, R41, R42, R43, R67, R69, R70, R71, R72, R73, R74, R89, R90, R91, R92: footprint sdi-mipi-bridge-footprints:0402-res -> antmicro-footprints:R_0402_1005Metric; symbol sdi-mipi-bridge:R_0R_0402 -> antmicroResistors0402:R_0R_0402
- R17, R18, R19, R20, R27, R28: footprint sdi-mipi-bridge-footprints:0603-res -> antmicro-footprints:R_0603_1608Metric; symbol sdi-mipi-bridge:R_75R_0603 -> antmicroResistors0603:R_75R_0603
- R29: footprint sdi-mipi-bridge-footprints:0402-res -> antmicro-footprints:R_0402_1005Metric; symbol sdi-mipi-bridge:R_37R4_0402 -> antmicroResistors0402:R_37R4_0402
- R30: footprint sdi-mipi-bridge-footprints:0402-res -> antmicro-footprints:R_0402_1005Metric; symbol sdi-mipi-bridge:R_105R_0402 -> antmicroResistors0402:R_105R_0402
- R33, R64, R88, R93: footprint sdi-mipi-bridge-footprints:0402-res -> antmicro-footprints:R_0402_1005Metric; symbol sdi-mipi-bridge:R_100R_0402 -> antmicroResistors0402:R_100R_0402
- R35, R36, R95: footprint sdi-mipi-bridge-footprints:0402-res -> antmicro-footprints:R_0402_1005Metric; symbol sdi-mipi-bridge:R_4k7_0402 -> antmicroResistors0402:R_4k7_0402
- R4: footprint sdi-mipi-bridge-footprints:0402-res -> antmicro-footprints:R_0402_1005Metric; symbol sdi-mipi-bridge:R_750R_0402 -> antmicroResistors0402:R_750R_0402
- R5, R6: footprint sdi-mipi-bridge-footprints:0402-res -> antmicro-footprints:R_0402_1005Metric; symbol sdi-mipi-bridge:R_120k_0402 -> antmicroResistors0402:R_120k_0402
- R85, R86, R87, R94: footprint sdi-mipi-bridge-footprints:0402-res -> antmicro-footprints:R_0402_1005Metric; symbol sdi-mipi-bridge:R_2k2_0402 -> antmicroResistors0402:R_2k2_0402
- R96: footprint sdi-mipi-bridge-footprints:0402-res -> antmicro-footprints:R_0402_1005Metric; symbol sdi-mipi-bridge:R_30R_0402 -> antmicroResistors0402:R_30R_0402
- S1: footprint sdi-mipi-bridge-footprints:Switch_Tactile_SMD_B3U-1000P -> antmicro-footprints:SW_B3U-3000P; symbol sdi-mipi-bridge:B3U-1000P -> antmicroTactileSwitches:SW_B3U-1000P
- TP1, TP17, TP18, TP19, TP2, TP20, TP21, TP6: footprint sdi-mipi-bridge-footprints:Testpoint_smd_1mm -> antmicro-footprints:Testpoint_smd_1mm; symbol sdi-mipi-bridge:TP_SMD1MM -> antmicroTestPoints:TP_1mm_SMD
- TP10, TP11, TP12, TP13, TP14, TP15, TP16, TP7, TP8, TP9: footprint sdi-mipi-bridge-footprints:Testpoint_smd_0_75mm -> antmicro-footprints:TP_SMD_0.75mm; symbol sdi-mipi-bridge:TP_SMD_0_75MM -> antmicroTestPoints:TP_0.75mm_SMD
- U1: footprint sdi-mipi-bridge-footprints:TDFN2x2 -> antmicro-footprints:TDFN2x2; symbol sdi-mipi-bridge:MAX8902B -> antmicroPMICVoltageRegulatorsLinear:MAX8902B
- U2: footprint sdi-mipi-bridge-footprints:BGA100_11x11mm -> antmicro-footprints:BGA-100_11x11mm_Layout10x10_P1mm; symbol sdi-mipi-bridge:GS2971A -> antmicroInterfaceControllers:GS2971A
- U3: footprint sdi-mipi-bridge-footprints:QFN-16_EP_4x4_Pitch0.65mm -> antmicro-footprints:QFN-16_1EP_4x4mm_P0.65mm; symbol sdi-mipi-bridge:GS2988 -> antmicroInterfaceControllers:GS2988
- U4: footprint sdi-mipi-bridge-footprints:BGA-80pin_ckfBGA80_7.0x7.0mm -> antmicro-footprints:BGA-80pin_ckfBGA80_7.0x7.0mm; symbol sdi-mipi-bridge:CrossLink_LIF-MD6000-6JMG80I -> antmicroBGAchips:CrossLink_LIF-MD6000-6JMG80I
- U5: footprint sdi-mipi-bridge-footprints:SC18IS602B -> antmicro-footprints:TSSOP-16_4.4x5mm_P0.65mm; symbol sdi-mipi-bridge:SC18IS602BIPW -> antmicroInterfaceDriversReceiversTransceivers:SC18IS602BIPW
- Y1: footprint sdi-mipi-bridge-footprints:ABM7_OSC -> antmicro-footprints:Oscillator_SMD_Abracon_ABM7-2Pin_6x3.5mm; symbol sdi-mipi-bridge:ABM7_27.000MH_D2Y_T -> antmicroOscillators:Oscillator_SMD_27MHz_ABM7

Commit message: Standardized SDI input and output sections
Parts:
- C18, C22, C36, C65: Author (none) -> Antmicro; Dielectric (none) -> X7R; License (none) -> Apache-2.0; MPN 04025G103ZAT2A -> GRM155R71H103KA88D; Manufacturer AVX -> Murata; Voltage (none) -> 50V
- C23, C31: Author (none) -> Antmicro; License (none) -> Apache-2.0; MPN GRM155R60G475ME -> GRM155R61A475MEAAD; Manufacturer MURATA -> Murata
- C27: Author (none) -> Antmicro; License (none) -> Apache-2.0; MPN C0402C562K3RACTU -> MC0402B562K160CT; Manufacturer Kemet -> Multicomp
- C39, C40, C41, C44, C46, C48, C49, C50, C51, C53, C54, C57: value C_100n_0402_6V3 -> C_100n_6V3_0402
- C43: Author (none) -> Antmicro; License (none) -> Apache-2.0; Manufacturer Kemet -> KEMET
- C55, C56, U3: Author (none) -> Antmicro; License (none) -> Apache-2.0
- D1, D2, D4, D5: value LG_L29K-G2J1-24-Z -> LED_G_0603_LG_L29K-G2J1-24-Z
- FB1, FB2, FB3: footprint antmicro-footprints:FB_0603_1608Metric -> sdi-mipi-bridge-footprints:0603-res
- J1, J2: value 112740-13 -> Conn_BNC_031-70526-21; Author (none) -> Antmicro; License (none) -> Apache-2.0; MPN 112740-13 -> 031-70526-21
- J3: value WE_68715014522_ONE-SIDE -> Conn_FFC_68715014522_ONE-SIDE
- J4: value GRPB052VWVN-RC -> 2199SB-10G-301523; MPN GRPB052VWVN-RC -> 2199SB-10G-301523; Manufacturer Sullins -> Multicomp
- J5: footprint antmicro-footprints:PinHeader_1x4_P1.27mm_Drill.7mm -> sdi-mipi-bridge-footprints:PinHeader_1x4_P1.27mm_Drill.7mm
- J6: footprint antmicro-footprints:PinHeader_2x05_P1.27mm_Vertical -> sdi-mipi-bridge-footprints:PinHeader_2x05_P1.27mm_Vertical
- R17, R18, R19, R20, R27, R28: Author (none) -> Antmicro; License (none) -> Apache-2.0; MPN RC0603FR-0775RL -> CR0603-FX-75R0ELF; Manufacturer Yageo -> Bourns; Tolerance (none) -> 1%
- R29: Author (none) -> Antmicro; License (none) -> Apache-2.0; MPN RC0402FR-0737R4L -> CR0402-FX-37R4GLF; Manufacturer Yageo -> Bourns; Tolerance (none) -> 1%
- R4: Author (none) -> Antmicro; License (none) -> Apache-2.0; MPN RC0402FR-07750RL -> CR0402-FX-7500GLF; Manufacturer Yageo -> Bourns; Tolerance (none) -> 1%
- R71: Author (none) -> Antmicro; Current (none) -> 1A; License (none) -> Apache-2.0; Manufacturer PANASONIC -> Panasonic
- R82: footprint antmicro-footprints:0402-res -> antmicro-footprints:R_0402_1005Metric
- S1: value B3U-1000P -> SW_B3U-1000P
- TP1, TP17, TP19, TP2, TP20, TP21, TP6: value TP_SMD1MM -> TP_1mm_SMD
- TP10, TP11, TP12, TP13, TP14, TP15, TP16, TP7, TP8, TP9: value TP_SMD_0_75MM -> TP_0.75mm_SMD
- TP18: value TP_SMD1MM -> TP_1mm_SMD; Author (none) -> Antmicro; License (none) -> Apache-2.0
- Y1: value ABM7_27.000MH_D2Y_T -> Oscillator_SMD_27MHz_ABM7
Connections:
- net GNDA: now also C18.1, C22.1, C36.2, C65.2, J1.2, J2.2; no longer C18.2, C22.2, C36.1, C65.1, J1.1 (In), J2.1 (In)
- net SDI_N: now also C56.2; no longer C56.1
- net SDI_P: now also C55.2; no longer C55.1
- net VDD: no longer C18.1, C22.1, C36.2, C65.2, R18.2, R19.2, R4.1, R71.1, U3.9 (VCC)
- net at R27.1, R28.1: now also C43.2, C55.1; no longer C43.1, C55.2
- net at R29.1: now also C56.1; no longer C56.2
- net at R17.1, U3.11 (SDO-): now also C27.1, R19.1; no longer C27.2, R18.1
- net at U3.13 (NC): now also U3.15 (NC), U3.5 (NC), U3.7 (NC), U3.8 (NC)
- net at C31.1: now also C27.2, R17.2; no longer J1.2 (Ext)
- net at C23.2: now also R18.1, U3.12 (SDO+); no longer R20.2
- new net: C43.1, J2.1, R27.2
- new net: C31.2, J1.1
- new net: C23.1, R20.2
- new net CD_VDD: C18.2, C22.2, C36.1, C65.1, R18.2, R19.2, R4.1, R71.1, U3.9 (V_{CC})
Other:
- moved on the sheet: C18, C22, C23, C27, C31, C36, C43, C55, C56, C58, C65, J1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

Commit message: Started standardizing the schematic
Parts:
- C11, C12, C13, C14, C16, C17, C19, C2, C20, C21, C3, C32, C33, C34, C4, C5, C6, C7, C8, C9: Author (none) -> Antmicro; Dielectric (none) -> X7R; License (none) -> Apache-2.0; MPN 04025G103ZAT2A -> GRM155R71H103KA88D; Manufacturer AVX -> Murata; Voltage (none) -> 50V
- C24, C25, C26, C28, C29, C30, C35, C59, C60, C61, C62, C64, TP10, TP11, TP12, TP13, TP14, TP15, TP16, TP17, TP7, TP8, TP9, U2, U5, Y1: Author (none) -> Antmicro; License (none) -> Apache-2.0
- C58: Author (none) -> Antmicro; License (none) -> Apache-2.0; Manufacturer Avx -> AVX
- C63: Author (none) -> Antmicro; License (none) -> Apache-2.0; MPN CGA2B2X7R1C473K050BA -> MC0402X473K160CT; Manufacturer TDK -> Multicomp
- J3: Author (none) -> Antmicro; License (none) -> Apache-2.0; MPN 68715014522 -> 68715014522; Manufacturer Wurth Elektronik -> Würth Elektronik
- R1, R2, R3: Author (none) -> Antmicro; License (none) -> Apache-2.0; MPN CRCW040222R0FKED -> CR0402-FX-22R0GLF; Manufacturer VISHAY -> Bourns; Tolerance (none) -> 1%
- R105, R21, R22, R23, R24, R25, R32, R34, R37, R38, R39, R40, R43, R67, R72, R73, R74, R92: Author (none) -> Antmicro; Current (none) -> 1A; License (none) -> Apache-2.0; Manufacturer PANASONIC -> Panasonic
- R30: Author (none) -> Antmicro; License (none) -> Apache-2.0; MPN RC0402FR-07105RL -> CR0402-FX-1050GLF; Manufacturer Yageo -> Bourns; Tolerance (none) -> 1%
- R41, R42: Author (none) -> Antmicro; Current (none) -> 1A; DNP DNP -> (none); License (none) -> Apache-2.0; Manufacturer PANASONIC -> Panasonic
- R84, R98: Author (none) -> Antmicro; License (none) -> Apache-2.0; MPN CRCW040210K0FKEDHP -> CR0402-FX-1002GLF; Manufacturer VISHAY -> Bourns; Tolerance (none) -> 1%
- R85, R86, R87, R94: Author (none) -> Antmicro; DNP DNP -> (none); License (none) -> Apache-2.0; MPN RC0402FR-072K2L -> CR0402-FX-2201GLF; Manufacturer YAGEO -> Bourns; Tolerance (none) -> 1%
Connections:
- net +1V2: now also C2.2, C20.2, C25.2, C4.2, C6.2, C8.2; no longer C2.1, C20.1, C25.1, C4.1, C6.1, C8.1
- net +3.3VA: now also C12.2, C14.2, C17.2, C28.2, C32.2; no longer C12.1, C14.1, C17.1, C28.1, C32.1
- net +3V3: now also C19.2, C21.2, C24.2, C26.2; no longer C19.1, C21.1, C24.1, C26.1
- net AGCN: now also C64.1; no longer C64.2
- net AGCP: now also C64.2; no longer C64.1
- net GNDA: now also C11.1, C12.1, C13.1, C14.1, C16.1, C17.1, C28.1, C29.1, C30.1, C32.1, C33.1, C34.1, C62.2, C63.2; no longer C11.2, C12.2, C13.2, C14.2, C16.2, C17.2, C28.2, C29.2, C30.2, C32.2, C33.2, C34.2, C62.1, C63.1
- net GNDREF: now also C19.1, C2.1, C20.1, C21.1, C24.1, C25.1, C26.1, C3.1, C35.1, C4.1, C5.1, C59.1, C6.1, C60.1, C7.1, C8.1, C9.1, J3.SH, R72.2, R73.2, R74.2; no longer C19.2, C2.2, C20.2, C21.2, C24.2, C25.2, C26.2, C3.2, C35.2, C4.2, C5.2, C59.2, C6.2, C60.2, C7.2, C8.2, C9.2, R72.1, R73.1, R74.1
- net IO_VDD: now also C3.2, C35.2, C5.2, C7.2, C9.2; no longer C3.1, C35.1, C5.1, C7.1, C9.1
- net LF: now also C63.1; no longer C63.2
- net VBG: now also C62.1; no longer C62.2
- net VDD: now also C30.2, C34.2; no longer C30.1, C34.1
- net VPP: now also C11.2, C13.2, C16.2, C29.2, C33.2; no longer C11.1, C13.1, C16.1, C29.1, C33.1, R30.1, U2.B2 (PLL_VDD), U2.C3 (PLL_VDD), U2.C4 (PLL_VDD)
- net XTAL1: now also C60.2; no longer C60.1
- net XTAL2: now also C59.2; no longer C59.1
- net at U2.B3 (RSV): now also U2.F2 (RSV)
- net at U5.14 (A0): now also R72.1; no longer R72.2
- net at U5.15 (A1): now also R73.1; no longer R73.2
- net at U5.16 (A2): now also R74.1; no longer R74.2
- new net +1.2VA: R30.1, U2.B2 (PLL_{VDD}), U2.C3 (PLL_{VDD}), U2.C4 (PLL_{VDD})
- no-connect marks 4 -> 21
Other:
- moved on the sheet: C11, C12, C13, C14, C16, C17, C19, C2, C20, C21, C24, C25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

Commit message: Continued schematic standarization
Parts:
- C37, C38: Author (none) -> Antmicro; License (none) -> Apache-2.0; MPN C0402C225K9PACTU -> C1005X5R1A225K050BC; Manufacturer Kemet -> TDK
- C39, C40, C41, C44, C45, C46, C47, C48, C49, C50, C51, C53, C54, C57, N1, N2: Author (none) -> Antmicro; License (none) -> Apache-2.0
- C42, C52: Author (none) -> Antmicro; License (none) -> Apache-2.0; MPN GRM155R60G475ME -> GRM155R61A475MEAAD; Manufacturer MURATA -> Murata
- D1, D2, D4, D5: Author (none) -> Antmicro; License (none) -> Apache-2.0; Manufacturer OSRAM Opto Semiconductors Inc. -> Osram
- FB1, FB2, FB3: footprint sdi-mipi-bridge-footprints:0603-res -> antmicro-footprints:FB_0603_1608Metric; Author (none) -> Antmicro; License (none) -> Apache-2.0; MPN BLM18PG121SH1D -> BLM18PG121SN1D; Manufacturer Murata Electronics North America -> Murata
- R100, R101, R102, R103, R104, R106, R107, R108, R109, R110, R111, R65, R66, R68, R75, R76, R77, R78, R79, R80, R81, R83, R97, R99: Author (none) -> Antmicro; License (none) -> Apache-2.0; MPN CRCW040210K0FKEDHP -> CR0402-FX-1002GLF; Manufacturer VISHAY -> Bourns; Tolerance (none) -> 1%
- R26, R31, R69, R70, R82: Author (none) -> Antmicro; Current (none) -> 1A; License (none) -> Apache-2.0; Manufacturer PANASONIC -> Panasonic
- R33, R64, R88, R93: Author (none) -> Antmicro; License (none) -> Apache-2.0; Manufacturer BOURNS -> Bourns; Tolerance (none) -> 1%
- S1: Author (none) -> Antmicro; License (none) -> Apache-2.0; Manufacturer Omron Electronics Inc-EMC Div -> Omron Electronics
Connections:
- net +1V2: now also C39.2, C42.2, C48.2, C52.2, FB3.2; no longer C39.1, C42.1, C48.1, C52.1, FB3.1
- net GNDGPLL: now also C47.1, C51.1; no longer C47.2, C51.2
- net GNDPLL_DPHY: now also C49.1, C53.1; no longer C49.2, C53.2
- net GNDREF: now also C37.1, C38.1, C39.1, C40.1, C41.1, C42.1, C44.1, C45.1, C46.1, C48.1, C50.1, C52.1, C54.1, C57.1; no longer C37.2, C38.2, C39.2, C40.2, C41.2, C42.2, C44.2, C45.2, C46.2, C48.2, C50.2, C52.2, C54.2, C57.2
- net VCCA_DPHY: now also C38.2, C40.2, C44.2, C49.2, C53.2; no longer C38.1, C40.1, C44.1, C49.1, C53.1
- net VCCGPLL: now also C47.2, C51.2, FB3.1; no longer C47.1, C51.1, FB3.2
- net VCC_IO: now also C37.2, C41.2, C46.2, C50.2, C54.2, C57.2; no longer C37.1, C41.1, C46.1, C50.1, C54.1, C57.1
- net at R26.2: now also C45.2; no longer C45.1
Other:
- moved on the sheet: C37, C38, C39, C40, C41, C42, C44, C45, C46, C47, C48, C49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

Commit message: Finished schematic migration
Parts:
- removed J4: 2199SB-10G-301523, antmicro-footprints:PinHeader_2x05_P1.27mm_Vertical, symbol antmicroRectangularConnectorsHeadersMalePins:2199SB-10G-301523
- removed J5: GRPB041VWVN-RC, sdi-mipi-bridge-footprints:PinHeader_1x4_P1.27mm_Drill.7mm, symbol antmicroRectangularConnectorsHeadersMalePins:MC-HVT1-S04-G
- removed J6: GRPB052VWVN-RC, sdi-mipi-bridge-footprints:PinHeader_2x05_P1.27mm_Vertical, symbol antmicroRectangularConnectorsHeadersMalePins:2199SB-10G-301523
- added J4, J6: PinHeader_2x5_P1.27mm_Vertical, antmicro-footprints:PinHeader_2x05_P1.27mm_Vertical, symbol antmicroRectangularConnectorsHeadersMalePins:PinHeader_2x5_P1.27mm_Vertical
- added J5: PinHeader_1x4_P1.27mm_Drill.7mm, antmicro-footprints:PinHeader_1x4_P1.27mm_Drill.7mm, symbol antmicroRectangularConnectorsHeadersMalePins:PinHeader_1x4_P1.27mm_Drill.7mm
- C1, C15: Author (none) -> Antmicro; License (none) -> Apache-2.0; MPN 06036D106MAT2A -> GRM188R61A106KE69D; Manufacturer AVX -> Murata
- C10: Author (none) -> Antmicro; Dielectric (none) -> X7R; License (none) -> Apache-2.0; MPN 04025G103ZAT2A -> GRM155R71H103KA88D; Manufacturer AVX -> Murata; Voltage (none) -> 50V
- R35, R36, R95: Author (none) -> Antmicro; License (none) -> Apache-2.0; MPN ERJ2GEJ472X -> CR0402-FX-4701GLF; Manufacturer PANASONIC_ELECTRONIC_COMPONENTS -> Bourns; Tolerance (none) -> 1%
- R5, R6: Author (none) -> Antmicro; License (none) -> Apache-2.0; MPN RC0402FR-07120KL -> CR0402-FX-1203GLF; Manufacturer Yageo -> Bourns; Tolerance (none) -> 1%
- R89: Author (none) -> Antmicro; Current (none) -> 1A; DNP DNP -> (none); License (none) -> Apache-2.0; Manufacturer PANASONIC -> Panasonic
- R90, R91: Author (none) -> Antmicro; Current (none) -> 1A; License (none) -> Apache-2.0; Manufacturer PANASONIC -> Panasonic
- R96: Author (none) -> Antmicro; License (none) -> Apache-2.0; MPN ERJ2GEJ300X -> CR0402-FX-30R0GLF; Manufacturer Panasonic -> Bourns; Tolerance (none) -> 1%
- TP1, TP19, TP2, TP20, TP21, TP6: Author (none) -> Antmicro; License (none) -> Apache-2.0
- U1: footprint antmicro-footprints:TDFN2x2 -> antmicro-footprints:TDFN-8-1EP_2x2mm_P0.5mm; Author (none) -> Antmicro; License (none) -> Apache-2.0
- U4: Author (none) -> Antmicro; License (none) -> Apache-2.0; Manufacturer Lattice Semiconductor -> Lattice; Manufacurer Lattice Semiconductor -> (none)
Connections:
- net +1V2: now also C10.2, C15.2; no longer C10.1, C15.1
- net +3V3: now also C1.2, J5.1, J6.1; no longer C1.1
- net AUDIO_MASTER_CLK: now also J4.10
- net AUDIO_OUTPUT_CH1_2: now also J4.5
- net AUDIO_OUTPUT_CH3_4: now also J4.7
- net AUDIO_OUTPUT_CH5_6: now also J4.6
- net AUDIO_OUTPUT_CH7_8: now also J4.8
- net AUDIO_SERIAL_BIT_CLK: now also J4.1, J4.2
- net AUDIO_WORD_CLK: now also J4.3, J4.4
- net CRESET_B: now also J6.8
- net GNDA: now also J4.9
- net GNDREF: now also C1.1, C15.1, U1.9 (EP), J5.4, J6.10; no longer C1.2, C15.2, U1.~ (EP)
- net MISO: now also J6.7
- net MOSI: now also J6.5
- net SCL_GS: now also J5.3
- net SDA_GS: now also J5.2
- net SPI_SCK(SDA): now also J6.3
- net SPI_SS(SCL): now also J6.9
- net USER_SCL: now also J6.4
- net USER_SDA: now also J6.2
- net at U1.7 (BYP): now also C10.1; no longer C10.2
Other:
- moved on the sheet: C1, C10, C15, R96, TP1, TP19, TP2, TP20, TP21, TP6

Commit message: Started migrating the PCB
Parts:
- N1: footprint antmicro-footprints:antmicro-logo -> antmicro-footprints:antmicro-logo_scaled_20mm
